Commit message: New Back-up with ICARUS_2c as working file, and ICARUS_2b beeing acceptable

File: rotors_simulator/rotors_description/urdf/ICARUS_2b.xacro (robot description, xacro)
@@ -26,7 +26,7 @@
   <xacro:property name="mass_elevator" value="0.05" /> <!-- [kg] 0.022-->
   <!-- Aileron properties -->
-  <xacro:property name="aileron_length" value="0.09" /> <!-- [m] 0.03-->
-  <xacro:property name="aileron_width" value="0.185" /> <!-- [m] 0.15-->
-  <xacro:property name="aileron_height" value="0.03" /> <!-- [m] 0.01-->
+  <xacro:property name="aileron_length" value="0.09" /> <!-- [m] -->
+  <xacro:property name="aileron_width" value="0.185" /> <!-- [m] -->
+  <xacro:property name="aileron_height" value="0.03" /> <!-- [m] -->
   <!-- <xacro:property name="aileron_min_angle" value="-0.349066" />  [rad] -->
   <!-- <xacro:property name="aileron_max_angle" value="0.349066" />  [rad]  -->
@@ -48,6 +48,5 @@
   <!-- Inertia of the elevator, assuming it is a cuboid -->
   <xacro:property name="elevator_inertia">
-    <xacro:box_inertia x="0.1" y="0.4" z="0.01" mass="${mass_elevator}"/> <!--Changed-->
-	<!-- <xacro:box_inertia x="${elevator_length}" y="${elevator_width}" z="${elevator_height}" mass="${mass_elevator}" />  -->
+	<xacro:box_inertia x="${elevator_length}" y="${elevator_width}" z="${elevator_height}" mass="${mass_elevator}" />
   </xacro:property>
   <!-- Servo PD controller paramters, tune after inertias of actuated links are set -->
@@ -68,6 +67,4 @@
   </xacro:property>
   <xacro:property name="distance_origin_ground" value="0.0" />
-  <xacro:property name="ram_eff" value="0.5" />
-  <xacro:property name="slip_eff" value="0.5" />
   <xacro:include filename="$(find rotors_description)/urdf/fixed_wing_X_base.xacro" />
   <!-- Fuselage -->
@@ -75,5 +72,5 @@
       <inertial>
         <mass value="0.3" /> <!--changed from 0.8 -->
-        <inertia ixx="0.0035" ixy="0.0" ixz="0.01" iyy="0.0082" iyz="0.0" izz="0.0045" />
+	<inertia ixx="0.0035" ixy="0.0" ixz="0.01" iyy="0.0082" iyz="0.0" izz="0.0045" />
         <origin xyz="0 0 0" rpy="0 0 0" />
       </inertial>
@@ -140,6 +137,4 @@
     <inertial>
       <mass value="0.1" />
-      <!--<inertia ixx="0.01" ixy="0.0" ixz="0.01" iyy="0.0" iyz="0.0" izz="0.01" />
-      <origin xyz="0 -0.060 0" rpy="0 0 0" /> -->
       <inertia ixx="0.0273" ixy="0.0" ixz="0.0002" iyy="0.0009" iyz="0.0" izz="0.0278" />
       <origin xyz="0 0 0" rpy="0 0 0" />
@@ -154,5 +149,5 @@
         <origin xyz="-0.05 0.25 0" rpy="0 0 0" />
         <geometry>
-          <box size="0.05 0.35 0.01" />
+          <box size="0.1 0.35 0.01" />
         </geometry>
     </collision>
@@ -172,6 +167,4 @@
       <inertial>
         <mass value="0.1" />
-        <!-- <inertia ixx="0.01" ixy="0.0" ixz="0.01" iyy="0.0" iyz="0.0" izz="0.01" />
-        <origin xyz="0 0.060 0" rpy="0 0 0" /> -->
         <inertia ixx="0.0273" ixy="0.0" ixz="0.0002" iyy="0.0009" iyz="0.0" izz="0.0278" />
         <origin xyz="0 0 0" rpy="0 0 0" />
@@ -186,5 +179,5 @@
         <origin xyz="-0.05 -0.25 0" rpy="0 0 0" />
         <geometry>
-          <box size="0.05 0.35 0.01" />
+          <box size="0.1 0.35 0.01" />
         </geometry>
     </collision>
@@ -241,5 +234,5 @@
   <joint name="${namespace}/elevator_joint" type="revolute">
     <origin xyz="-0.465 0 0.0" rpy="0 0 0" />
-    <axis xyz="0 1 0" />
+    <axis xyz="0 -1 0" />
     <parent link="${namespace}/base_link" />
     <child link="${namespace}/elevator" />
@@ -343,33 +336,4 @@
     <material>Gazebo/Orange</material>
   </gazebo>
-  <!--
-  <joint name="${namespace}/propeller_back_right_joint" type="continuous">
-    <origin xyz="0.0 -0.185 0" rpy="0 ${0.5*pi} 0" />
-    <axis xyz="0 0 1" />
-    <parent link="${namespace}/elevator" />
-    <child link="${namespace}/propeller_back_right" />
-  </joint>
-  <link name="${namespace}/propeller_back_right">
-    <inertial>
-      <mass value="0.01" />
-      <xacro:cylinder_inertia r="0.08" h="0.01" mass="0.01" />
-    </inertial>
-    <visual>
-      <origin xyz="0 0 0.04" rpy="0 0 0" />
-      <geometry>
-        <mesh filename="package://rotors_description/meshes/IGNIS/ICARUS_2/iris_prop_ccw.dae" scale="0.6 0.6 0.6"/>
-      </geometry>
-    </visual>
-    <visual>
-      <origin xyz="0 0 0.03" rpy="0 0 0" />
-      <geometry>
-        <cylinder radius="0.01" length="0.01" />
-      </geometry>
-    </visual>
-  </link>
-  <gazebo reference="${namespace}/propeller_back_right">
-    <material>Gazebo/Orange</material>
-  </gazebo>
-  -->
   <!-- propeller plugin -->
   <gazebo>
@@ -380,13 +344,12 @@
         <linkNameAct>${namespace}/base_link</linkNameAct>
         <cp>0.080 0.140 -0.010</cp>			<!-- !!! -->
-        <axisPosRot>-0.9877 0 -0.1564</axisPosRot>
+        <axisPosRot>-1 0 0</axisPosRot>
         <turnDir>cw</turnDir>
         <speedRefTopic>propeller_front_left_ref</speedRefTopic>
-        <propParamsYAML>${yaml_path}/cl84b_main_prop.yaml</propParamsYAML>
+        <propParamsYAML>${yaml_path}/ic2_main_prop.yaml</propParamsYAML>
         <tauUp>0.075</tauUp>
         <tauDown>0.15</tauDown>
         <rdpsMax>2039</rdpsMax>
         <slpstrTopic>propeller_front_left_slpstr</slpstrTopic>
-        <ramEff>${ram_eff}</ramEff>
         <visTopic>propeller_front_left_vis</visTopic>
         <wind name="wind">
@@ -398,13 +361,12 @@
         <linkNameAct>${namespace}/base_link</linkNameAct>
         <cp>0.080 -0.140 -0.010</cp>
-        <axisPosRot>0.9877 0 0.1564</axisPosRot>
+        <axisPosRot>1 0 0</axisPosRot>
         <turnDir>ccw</turnDir>
         <speedRefTopic>propeller_front_right_ref</speedRefTopic>
-        <propParamsYAML>${yaml_path}/cl84b_main_prop.yaml</propParamsYAML>
+        <propParamsYAML>${yaml_path}/ic2_main_prop.yaml</propParamsYAML>
         <tauUp>0.075</tauUp>
         <tauDown>0.15</tauDown>
         <rdpsMax>2039</rdpsMax>
         <slpstrTopic>propeller_front_right_slpstr</slpstrTopic>
-        <ramEff>${ram_eff}</ramEff>
         <visTopic>propeller_front_right_vis</visTopic>
         <wind name="wind">
@@ -419,10 +381,9 @@
         <turnDir>ccw</turnDir>
         <speedRefTopic>propeller_back_ref</speedRefTopic>
-        <propParamsYAML>${yaml_path}/cl84b_tail_prop.yaml</propParamsYAML>
+        <propParamsYAML>${yaml_path}/cl84_tail_prop.yaml</propParamsYAML>
         <tauUp>0.05</tauUp>
         <tauDown>0.1</tauDown>
-	<rdpsMax>5183</rdpsMax>
+	<rdpsMax>5183</rdpsMax> <!-- !!!!!!!!!!!!!!!!!!!!!!!!!!!!!! -->
         <slpstrTopic>propeller_back_slpstr</slpstrTopic>
-        <ramEff>${ram_eff}</ramEff>
         <visTopic>propeller_back_vis</visTopic>
         <wind name="wind">
@@ -430,24 +391,4 @@
         </wind>
       </prop>
-<!--
-      <prop name="propeller_back_right">
-        <linkNameRef>${namespace}/elevator</linkNameRef>
-        <linkNameAct>${namespace}/base_link</linkNameAct>
-        <cp>-0.03 0 0.04</cp>
-        <axisPosRot>0 0 1</axisPosRot>
-        <turnDir>ccw</turnDir>
-        <speedRefTopic>propeller_back_right_ref</speedRefTopic>
-        <propParamsYAML>${yaml_path}/cl84b_tail_prop.yaml</propParamsYAML>
-        <tauUp>0.05</tauUp>
-        <tauDown>0.1</tauDown>
-        <rdpsMax>1410</rdpsMax>
-        <slpstrTopic>propeller_back_right_slpstr</slpstrTopic>
-        <ramEff>${ram_eff}</ramEff>
-        <visTopic>propeller_back_right_vis</visTopic>
-        <wind name="wind">
-          <topic>wind_base_link</topic>
-        </wind>
-      </prop>
--->
     </plugin>
   </gazebo>
@@ -460,10 +401,10 @@
       <body>
         <element>
-          <aBdyXX>0.01125</aBdyXX>
-          <aBdyYY>0</aBdyYY>
-          <aBdyZZ>0</aBdyZZ>
+          <aBdyXX>0.012</aBdyXX>
+          <aBdyYY>0</aBdyYY>  <!-- 0.068 -->
+          <aBdyZZ>0</aBdyZZ> <!-- 0.077 -->
           <forward>1 0 0</forward>
           <upward>0 0 1</upward>
-          <cp>0.18 0.0 0.15</cp>
+	  <cp>0.0 0.0 0.0</cp>
           <wind name="wind">
             <topic>wind_base_link</topic>
@@ -473,5 +414,4 @@
     </plugin>
   </gazebo>
-<!-- Why is the y-axis pointing negatively towards convention? -->
   <!-- aft wing L&D plugin -->
   <gazebo>
@@ -485,15 +425,11 @@
           <forward>1 0 0</forward>
           <upward>0 0 1</upward>
-          <cp>-0.39 0.1 0.0</cp>
+          <cp>-0.03 0.1 0.0</cp>
           <seg_area>0.0112</seg_area>
           <seg_chord>0.08</seg_chord>
-          <aeroParamsYAML>${yaml_path}/cl84b_wing_airfoil.yaml</aeroParamsYAML>
+          <aeroParamsYAML>${yaml_path}/---ic2_wing_airfoil.yaml</aeroParamsYAML>
           <wind name="wind">
             <topic>wind_base_link</topic>
           </wind>
-          <!-- <indVel name="propeller_back">
-             <topic>propeller_back_slpstr</topic>
-             <eff>${slip_eff}</eff>
-          </indVel> -->
         </segment>
         <segment name="ER">
@@ -502,26 +438,12 @@
           <forward>1 0 0</forward>
           <upward>0 0 1</upward>
-          <cp>-0.39 -0.1 0.0</cp>
+          <cp>-0.03 -0.1 0.0</cp>
           <seg_area>0.0112</seg_area>
           <seg_chord>0.08</seg_chord>
-          <aeroParamsYAML>${yaml_path}/cl84b_wing_airfoil.yaml</aeroParamsYAML>
+          <aeroParamsYAML>${yaml_path}/---ic2_wing_airfoil.yaml</aeroParamsYAML>
           <wind name="wind">
             <topic>wind_base_link</topic>
           </wind>
-          <!-- <indVel name="propeller_back_right">
-             <topic>propeller_back_right_slpstr</topic>
-             <eff>${slip_eff}</eff>
-          </indVel> -->
         </segment>
-      </airfoil>
-    </plugin>
-  </gazebo>
-  <!-- horizontal stabilizer L&D plugin -->
-  <!--
-  <gazebo>
-    <plugin filename="librotors_gazebo_aerodynamics_plugin.so" name="aerodynamics_plugin">
-      <robotNamespace>${namespace}</robotNamespace>
-      <aeroForcesVis>aero_force_vis_1</aeroForcesVis>
-      <airfoil>
         <segment name="VS">
           <linkNameRef>${namespace}/base_link</linkNameRef>
@@ -529,5 +451,5 @@
           <forward>1 0 0</forward>
           <upward>0 1 0</upward>
-          <cp>-0.22 0 0.24</cp>
+          <cp>-0.41 0 0.1</cp>
           <seg_area>0.015</seg_area>
           <seg_chord>0.15</seg_chord>
@@ -540,5 +462,4 @@
     </plugin>
   </gazebo>
-  -->
   <!-- front wing L&D plugin -->
   <gazebo>
@@ -552,8 +473,8 @@
         <forward>1 0 0</forward>
         <upward>0 0 1</upward>
-        <cp>0.01 0.1100 -0.005</cp>
+        <cp>-0.05 0.0500 -0.005</cp>
         <seg_area>0.020</seg_area>
         <seg_chord>0.20</seg_chord>
-        <aeroParamsYAML>${yaml_path}/cl84b_wing_airfoil.yaml</aeroParamsYAML>
+        <aeroParamsYAML>${yaml_path}/---ic2_wing_airfoil.yaml</aeroParamsYAML>
         <wind name="wind">
           <topic>wind_base_link</topic>
@@ -565,8 +486,8 @@
         <forward>1 0 0</forward>
         <upward>0 0 1</upward>
-        <cp>0.01 0.2225 -0.005</cp>
+        <cp>-0.05 0.1625 -0.005</cp>
         <seg_area>0.025</seg_area>
         <seg_chord>0.20</seg_chord>
-        <aeroParamsYAML>${yaml_path}/cl84b_wing_airfoil.yaml</aeroParamsYAML>
+        <aeroParamsYAML>${yaml_path}/---ic2_wing_airfoil.yaml</aeroParamsYAML>
         <wind name="wind">
           <topic>wind_base_link</topic>
@@ -574,5 +495,4 @@
         <indVel name="propeller_front_left">
            <topic>propeller_front_left_slpstr</topic>
-           <eff>${slip_eff}</eff>
         </indVel>
       </segment>
@@ -582,12 +502,12 @@
         <forward>1 0 0</forward>
         <upward>0 0 1</upward>
-        <cp>0.01 0.3475 -0.005</cp>
+        <cp>-0.05 0.2875 -0.005</cp>
         <seg_area>0.025</seg_area>
         <seg_chord>0.20</seg_chord>
-        <aeroParamsYAML>${yaml_path}/cl84b_wing_airfoil.yaml</aeroParamsYAML>
+        <aeroParamsYAML>${yaml_path}/---ic2_wing_airfoil.yaml</aeroParamsYAML>
         <control>
           <cs name="aileron_left">
               <controlJoint>${namespace}/aileron_left_joint</controlJoint>
-              <radToCLift>2</radToCLift>
+              <radToCLift>3</radToCLift> <!-- !!!!!!!!!!!!!!!!! -->
               <radToCDrag>0.0</radToCDrag>
               <radToCPitch>0.0</radToCPitch>
@@ -599,5 +519,4 @@
         <indVel name="propeller_front_left">
            <topic>propeller_front_left_slpstr</topic>
-           <eff>${slip_eff}</eff>
         </indVel>
       </segment>
@@ -607,8 +526,8 @@
         <forward>1 0 0</forward>
         <upward>0 0 1</upward>
-        <cp>0.01 0.4550 -0.005</cp>
+        <cp>-0.05 0.3950 -0.005</cp>
         <seg_area>0.018</seg_area>
         <seg_chord>0.20</seg_chord>
-        <aeroParamsYAML>${yaml_path}/cl84b_wing_airfoil.yaml</aeroParamsYAML>
+        <aeroParamsYAML>${yaml_path}/---ic2_wing_airfoil.yaml</aeroParamsYAML>
         <wind name="wind">
           <topic>wind_base_link</topic>
@@ -617,5 +536,5 @@
           <cs name="aileron_left">
               <controlJoint>${namespace}/aileron_left_joint</controlJoint>
-              <radToCLift>2</radToCLift>
+              <radToCLift>3</radToCLift> <!-- !!!!!!!!!!!!!!!!!!!!!!! -->
               <radToCDrag>0.0</radToCDrag>
               <radToCPitch>0.0</radToCPitch>
@@ -628,8 +547,8 @@
         <forward>1 0 0</forward>
         <upward>0 0 1</upward>
-        <cp>0.01 -0.0110 -0.005</cp>
+        <cp>-0.05 -0.0500 -0.005</cp>
         <seg_area>0.020</seg_area>
         <seg_chord>0.20</seg_chord>
-        <aeroParamsYAML>${yaml_path}/cl84b_wing_airfoil.yaml</aeroParamsYAML>
+        <aeroParamsYAML>${yaml_path}/---ic2_wing_airfoil.yaml</aeroParamsYAML>
         <wind name="wind">
           <topic>wind_base_link</topic>
@@ -641,8 +560,8 @@
         <forward>1 0 0</forward>
         <upward>0 0 1</upward>
-        <cp>0.01 -0.2225 -0.005</cp>
+        <cp>-0.05 -0.1625 -0.005</cp>
         <seg_area>0.025</seg_area>
         <seg_chord>0.20</seg_chord>
-        <aeroParamsYAML>${yaml_path}/cl84b_wing_airfoil.yaml</aeroParamsYAML>
+        <aeroParamsYAML>${yaml_path}/---ic2_wing_airfoil.yaml</aeroParamsYAML>
         <wind name="wind">
           <topic>wind_base_link</topic>
@@ -650,5 +569,4 @@
         <indVel name="propeller_front_right">
            <topic>propeller_front_right_slpstr</topic>
-           <eff>${slip_eff}</eff>
         </indVel>
       </segment>
@@ -658,12 +576,12 @@
         <forward>1 0 0</forward>
         <upward>0 0 1</upward>
-        <cp>0.01 -0.3475 -0.005</cp>
+        <cp>-0.05 -0.2875 -0.005</cp>
         <seg_area>0.025</seg_area>
         <seg_chord>0.20</seg_chord>
-        <aeroParamsYAML>${yaml_path}/cl84b_wing_airfoil.yaml</aeroParamsYAML>
+        <aeroParamsYAML>${yaml_path}/---ic2_wing_airfoil.yaml</aeroParamsYAML>
         <control>
           <cs name="aileron_right">
               <controlJoint>${namespace}/aileron_right_joint</controlJoint>
-              <radToCLift>2</radToCLift>
+              <radToCLift>3</radToCLift> <!-- !!!!!!!!!!!!!!!!! -->
               <radToCDrag>0.0</radToCDrag>
               <radToCPitch>0.0</radToCPitch>
@@ -675,5 +593,4 @@
         <indVel name="propeller_front_right">
            <topic>propeller_front_right_slpstr</topic>
-           <eff>${slip_eff}</eff>
         </indVel>
       </segment>
@@ -683,8 +600,8 @@
         <forward>1 0 0</forward>
         <upward>0 0 1</upward>
-        <cp>0.01 -0.4550 -0.005</cp>
+        <cp>-0.05 -0.3950 -0.005</cp>
         <seg_area>0.018</seg_area>
         <seg_chord>0.20</seg_chord>
-        <aeroParamsYAML>${yaml_path}/cl84b_wing_airfoil.yaml</aeroParamsYAML>
+        <aeroParamsYAML>${yaml_path}/---ic2_wing_airfoil.yaml</aeroParamsYAML>
         <wind name="wind">
           <topic>wind_base_link</topic>
@@ -693,5 +610,5 @@
           <cs name="aileron_right">
               <controlJoint>${namespace}/aileron_right_joint</controlJoint>
-              <radToCLift>2</radToCLift>
+              <radToCLift>3</radToCLift> <!-- !!!!!!!!!!!!!!!!!!!!!!!!!! -->
               <radToCDrag>0.0</radToCDrag>
               <radToCPitch>0.0</radToCPitch>
@@ -736,5 +653,5 @@
           <input_index>0</input_index>
           <input_offset>1</input_offset>
-          <input_scaling>505</input_scaling>
+          <input_scaling>1016</input_scaling>
           <zero_position_disarmed>0</zero_position_disarmed>
           <zero_position_armed>0</zero_position_armed>
@@ -754,5 +671,5 @@
           <input_index>1</input_index>
           <input_offset>1</input_offset>
-          <input_scaling>505</input_scaling>
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