Commit message: New Back-up Icarus_2c should be working good enough, and Scintilla_01 is on its way to work

File: rotors_simulator/rotors_description/urdf/ICARUS_2c.xacro (robot description, xacro)
@@ -13,5 +13,5 @@
 -->
 <robot name="ICARUS_2c" xmlns:xacro="http://ros.org/wiki/xacro">
-  <!-- Global properties -->
+ <!-- Global properties -->
   <xacro:property name="namespace" value="$(arg namespace)" />
   <xacro:property name="rotor_velocity_slowdown_sim" value="10" />
@@ -29,6 +29,4 @@
   <xacro:property name="aileron_width" value="0.185" /> <!-- [m] -->
   <xacro:property name="aileron_height" value="0.03" /> <!-- [m] -->
-  <!-- <xacro:property name="aileron_min_angle" value="-0.349066" />  [rad] -->
-  <!-- <xacro:property name="aileron_max_angle" value="0.349066" />  [rad]  -->
   <xacro:property name="aileron_color" value="Red" />
   <xacro:property name="aileron_left_mesh_file" value="package://rotors_description/meshes/techpod/techpod_aileron_left.dae" />
@@ -37,7 +35,5 @@
   <xacro:property name="elevator_length" value="0.08" /> <!-- [m] -->
   <xacro:property name="elevator_width" value="0.4" /> <!-- [m] -->
-  <xacro:property name="elevator_height" value="0.01" /> <!-- [m] 0.05-->
-  <!-- <xacro:property name="elevator_min_angle" value="-0.349066" /> [rad] -->
-  <!-- <xacro:property name="elevator_max_angle" value="0.349066" /> [rad] -->
+  <xacro:property name="elevator_height" value="0.01" /> <!-- [m] -->
   <xacro:property name="elevator_color" value="Blue" />
   <xacro:property name="elevator_mesh_file" value="package://rotors_description/meshes/techpod/techpod_elevator.dae" />
@@ -48,5 +44,5 @@
   <!-- Inertia of the elevator, assuming it is a cuboid -->
   <xacro:property name="elevator_inertia">
-	<xacro:box_inertia x="${elevator_length}" y="${elevator_width}" z="${elevator_height}" mass="${mass_elevator}" />
+	  <xacro:box_inertia x="${elevator_length}" y="${elevator_width}" z="${elevator_height}" mass="${mass_elevator}" />
   </xacro:property>
   <!-- Servo PD controller paramters, tune after inertias of actuated links are set -->
@@ -63,18 +59,18 @@
   <xacro:property name="wing_srv_params">
     <slew>0.52</slew>
-    <p>5</p>
+    <p>20</p>
     <d>0</d>
   </xacro:property>
-  <xacro:property name="distance_origin_ground" value="0.0" />
   <xacro:include filename="$(find rotors_description)/urdf/fixed_wing_X_base.xacro" />
   <!-- Fuselage -->
   <link name="${namespace}/base_link">
       <inertial>
-        <mass value="0.3" /> <!--changed from 0.8 -->
-	<inertia ixx="0.0035" ixy="0.0" ixz="0.01" iyy="0.0082" iyz="0.0" izz="0.0045" />
-        <origin xyz="0 0 0" rpy="0 0 0" />
+        <origin xyz="-0.01 0 -0.025" rpy="0 0 0" /> <!-- CG has to be in these coordinates -->
+        <mass value="1.0" />
+        <inertia ixx="0.0033" ixy="0.0" ixz="0.0" iyy="0.0473" iyz="0.0" izz="0.0472" />
+        <!-- <xacro:box_inertia x="0.65" y="0.12" z="0.1" mass="1.0" /> -->
       </inertial>
       <visual>
-        <origin xyz="0 0 ${distance_origin_ground}" rpy="${pi/2} 0 ${pi}" />
+        <origin xyz="0 0 0" rpy="${pi/2} 0 ${pi}" />
         <geometry>
           <mesh filename="package://rotors_description/meshes/IGNIS/ICARUS_2/Fuselage.stl" scale="0.001 0.001 0.001" />
@@ -82,5 +78,11 @@
       </visual>
       <collision>
-        <origin xyz="0.1 -0.1 -0.1" rpy="0 0 0" />
+        <origin xyz="-0.1 0 -0.02" rpy="0 0 0" />
+        <geometry>
+          <box size="0.65 0.12 0.1" />
+        </geometry>
+      </collision>
+      <collision>
+        <origin xyz="0.1 -0.09 -0.1" rpy="0 0 0" />
         <geometry>
           <sphere radius="0.05" />
@@ -88,5 +90,5 @@
       </collision>
       <collision>
-        <origin xyz="0.1 0.1 -0.1" rpy="0 0 0" />
+        <origin xyz="0.1 0.09 -0.1" rpy="0 0 0" />
         <geometry>
           <sphere radius="0.05" />
@@ -103,26 +105,4 @@
     <material>Gazebo/White</material>
   </gazebo>
-<!-- Center of Gravity manipulation -->
-  <joint name="${namespace}/CG_joint" type="fixed">
-    <parent link="${namespace}/base_link" />
-    <child link="${namespace}/CG" />
-    <origin xyz="-0.1 0 -0.05" rpy="0 0 0" />
-  </joint>
-  <link name="${namespace}/CG">
-    <inertial>
-      <mass value="0.5" />
-      <inertia ixx="0.002" ixy="0.0" ixz="0.001" iyy="0.002" iyz="0.0" izz="0.001" />
-      <origin xyz="0 0 0" rpy="0 0 0" />
-    </inertial>
-    <visual>
-      <origin xyz="0 0 0" rpy="0 0 0" />
-      <geometry>
-        <cylinder radius="0.025" length="0.02" />
-      </geometry>
-    </visual>
-  </link>
-  <gazebo reference="${namespace}/CG">
-    <material>Gazebo/Black</material>
-  </gazebo>
   <!-- Wing -->
   <joint name="${namespace}/wing_left_joint" type="revolute">
@@ -132,24 +112,24 @@
     <axis xyz="0 1 0" />
     <limit upper="0.0" lower="-1.57" effort="10" velocity="20"/>
-    <dynamics damping="0.2" friction="0" />
+    <dynamics damping="0.1" friction="0" />
   </joint>
   <link name="${namespace}/wing_left">
     <inertial>
-      <mass value="0.1" />
-      <!-- <inertia ixx="0.0273" ixy="0.0" ixz="0.0002" iyy="0.0009" iyz="0.0" izz="0.0278" /> -->
-	<xacro:box_inertia x="0.20" y="0.44" z="0.02" mass="0.1" />
+      <mass value="0.2" />
+      <xacro:box_inertia x="0.2" y="0.44" z="0.02" mass="0.2" />
+      <!--<origin xyz="-0.1 0.22 0" rpy="0 0 0" />-->
+      <origin xyz="0 0.22 0" rpy="0 0 0" />
+    </inertial>
+    <visual>
+      <origin xyz="0.05 0.500 0" rpy="${pi/2} 0 ${pi}" />
+      <geometry>
+        <mesh filename="package://rotors_description/meshes/IGNIS/ICARUS_2/Wing.stl" scale="0.001 0.001 0.001" />
+      </geometry>
+    </visual>
+    <collision>
       <origin xyz="-0.1 0.22 0" rpy="0 0 0" />
-    </inertial>
-    <visual>
-      <origin xyz="0 0.500 0" rpy="${pi/2} 0 ${pi}" />
-      <geometry>
-        <mesh filename="package://rotors_description/meshes/IGNIS/ICARUS_2/Wing.stl" scale="0.001 0.001 0.001" />
-      </geometry>
-    </visual>
-    <collision>
-        <origin xyz="-0.05 0.25 0" rpy="0 0 0" />
-        <geometry>
-          <box size="0.1 0.35 0.01" />
-        </geometry>
+      <geometry>
+        <box size="0.1 0.44 0.02" />
+      </geometry>
     </collision>
   </link>
@@ -167,11 +147,11 @@
   <link name="${namespace}/wing_right">
       <inertial>
-        <mass value="0.1" />
-      <!-- <inertia ixx="0.0273" ixy="0.0" ixz="0.0002" iyy="0.0009" iyz="0.0" izz="0.0278" /> -->
-	<xacro:box_inertia x="0.20" y="0.44" z="0.02" mass="0.1" />
-        <origin xyz="-0.1 -0.22 0" rpy="0 0 0" />
+        <mass value="0.2" />
+        <xacro:box_inertia x="0.2" y="0.44" z="0.02" mass="0.2" />
+        <!--<origin xyz="-0.1 -0.22 0" rpy="0 0 0" />-->
+        <origin xyz="0 -0.22 0" rpy="0 0 0" />
       </inertial>
       <visual>
-        <origin xyz="0 0.060 0" rpy="${pi/2} 0 ${pi}" />
+        <origin xyz="0.05 0.060 0" rpy="${pi/2} 0 ${pi}" />
         <geometry>
           <mesh filename="package://rotors_description/meshes/IGNIS/ICARUS_2/Wing.stl" scale="0.001 0.001 0.001" />
@@ -179,7 +159,7 @@
       </visual>
       <collision>
-        <origin xyz="-0.05 -0.25 0" rpy="0 0 0" />
+        <origin xyz="-0.1 -0.22 0" rpy="0 0 0" />
         <geometry>
-          <box size="0.1 0.35 0.01" />
+          <box size="0.1 0.44 0.02" />
         </geometry>
     </collision>
@@ -190,5 +170,5 @@
   <!-- Ailerons -->
   <joint name="${namespace}/aileron_left_joint" type="revolute">
-    <origin xyz="-0.1 0.355 -0.007" rpy="0 0 0" />
+    <origin xyz="-0.05 0.355 -0.007" rpy="0 0 0" />
     <axis xyz="0 -1 0" />
     <parent link="${namespace}/wing_left" />
@@ -200,4 +180,5 @@
       <mass value="${mass_aileron}" />
       <xacro:insert_block name="aileron_inertia" />
+      <!--<origin xyz="-0.045 0 0" rpy="0 0 0" />-->
     </inertial>
     <visual>
@@ -212,5 +193,5 @@
   </gazebo>
   <joint name="${namespace}/aileron_right_joint" type="revolute">
-    <origin xyz="-0.1 -0.355 -0.007" rpy="0 0 0" />
+    <origin xyz="-0.05 -0.355 -0.007" rpy="0 0 0" />
     <axis xyz="0 -1 0" />
     <parent link="${namespace}/wing_right" />
@@ -222,4 +203,5 @@
       <mass value="${mass_aileron}" />
       <xacro:insert_block name="aileron_inertia" />
+      <!--<origin xyz="-0.045 0 0" rpy="0 0 0" />-->
     </inertial>
     <visual>
@@ -243,7 +225,7 @@
   <link name="${namespace}/elevator">
     <inertial>
-      <origin xyz="-0.03 0.0 0" rpy="0 0 0" />
       <mass value="${mass_elevator}" />
       <xacro:insert_block name="elevator_inertia" />
+      <!-- <origin xyz="-0.04 0 0" rpy="0 0 0" /> -->
     </inertial>
     <visual>
@@ -259,5 +241,5 @@
   <!-- Propellers -->
   <joint name="${namespace}/propeller_front_left_joint" type="continuous">
-    <origin xyz="0.03 0.225 0" rpy="0 ${0.5*pi} 0" />
+    <origin xyz="0.08 0.225 0" rpy="0 ${0.5*pi} 0" />
     <axis xyz="0 0 1" />
     <parent link="${namespace}/wing_left" />
@@ -266,6 +248,7 @@
   <link name="${namespace}/propeller_front_left">
     <inertial>
-      <mass value="0.0125" />
-      <xacro:cylinder_inertia r="0.14" h="0.02" mass="0.0125" />
+      <mass value="0.1" />
+      <xacro:cylinder_inertia r="0.14" h="0.02" mass="0.1" />
+      <origin xyz="0 0 -0.03" rpy="0 0 0" />
     </inertial>
     <visual>
@@ -286,5 +269,5 @@
   </gazebo>
   <joint name="${namespace}/propeller_front_right_joint" type="continuous">
-    <origin xyz="0.03 -0.225 0" rpy="0 ${0.5*pi} 0" />
+    <origin xyz="0.08 -0.225 0" rpy="0 ${0.5*pi} 0" />
     <axis xyz="0 0 1" />
     <parent link="${namespace}/wing_right" />
@@ -293,6 +276,7 @@
   <link name="${namespace}/propeller_front_right">
     <inertial>
-      <mass value="0.0125" />
-      <xacro:cylinder_inertia r="0.14" h="0.02" mass="0.0125" />
+      <mass value="0.1" />
+      <xacro:cylinder_inertia r="0.14" h="0.02" mass="0.1" />
+      <origin xyz="0 0 -0.03" rpy="0 0 0" />
     </inertial>
     <visual>
@@ -320,5 +304,5 @@
   <link name="${namespace}/propeller_back">
     <inertial>
-      <mass value="0.1" /> <!-- 0.01 -->
+      <mass value="0.1" />
       <xacro:cylinder_inertia r="0.08" h="0.01" mass="0.01" />
     </inertial>
@@ -339,5 +323,5 @@
     <material>Gazebo/Orange</material>
   </gazebo>
-  <!-- propeller plugin -->
+  <!-- propeller plugins -->
   <gazebo>
     <plugin filename="librotors_gazebo_propulsion_plugin.so" name="propulsion_plugin">
@@ -346,5 +330,5 @@
         <linkNameRef>${namespace}/wing_left</linkNameRef>
         <linkNameAct>${namespace}/base_link</linkNameAct>
-        <cp>0.080 0.140 -0.010</cp>			<!-- !!! -->
+        <cp>0.08 0.225 0</cp>			<!-- !!! -->
         <axisPosRot>-1 0 0</axisPosRot>
         <turnDir>cw</turnDir>
@@ -353,5 +337,5 @@
         <tauUp>0.075</tauUp>
         <tauDown>0.15</tauDown>
-        <rdpsMax>2039</rdpsMax>
+        <rdpsMax>2040</rdpsMax>
         <slpstrTopic>propeller_front_left_slpstr</slpstrTopic>
         <visTopic>propeller_front_left_vis</visTopic>
@@ -363,5 +347,5 @@
         <linkNameRef>${namespace}/wing_right</linkNameRef>
         <linkNameAct>${namespace}/base_link</linkNameAct>
-        <cp>0.080 -0.140 -0.010</cp>
+        <cp>0.08 -0.225 0</cp>
         <axisPosRot>1 0 0</axisPosRot>
         <turnDir>ccw</turnDir>
@@ -370,5 +354,5 @@
         <tauUp>0.075</tauUp>
         <tauDown>0.15</tauDown>
-        <rdpsMax>2039</rdpsMax>
+        <rdpsMax>2040</rdpsMax>
         <slpstrTopic>propeller_front_right_slpstr</slpstrTopic>
         <visTopic>propeller_front_right_vis</visTopic>
@@ -380,12 +364,12 @@
         <linkNameRef>${namespace}/base_link</linkNameRef>
         <linkNameAct>${namespace}/base_link</linkNameAct>
-        <cp>-0.43,0,-0.02</cp>
+        <cp>-0.53 0 0</cp>
         <axisPosRot>0 0 1</axisPosRot>
         <turnDir>ccw</turnDir>
         <speedRefTopic>propeller_back_ref</speedRefTopic>
-        <propParamsYAML>${yaml_path}/cl84_tail_prop.yaml</propParamsYAML>
+        <propParamsYAML>${yaml_path}/ic2_tail_prop.yaml</propParamsYAML>
         <tauUp>0.05</tauUp>
         <tauDown>0.1</tauDown>
-	<rdpsMax>5183</rdpsMax> <!-- !!!!!!!!!!!!!!!!!!!!!!!!!!!!!! -->
+	      <rdpsMax>5180</rdpsMax>
         <slpstrTopic>propeller_back_slpstr</slpstrTopic>
         <visTopic>propeller_back_vis</visTopic>
@@ -404,10 +388,10 @@
       <body>
         <element>
-          <aBdyXX>0.012</aBdyXX>
-          <aBdyYY>0</aBdyYY>  <!-- 0.068 -->
-          <aBdyZZ>0</aBdyZZ> <!-- 0.077 -->
-          <forward>1 0 0</forward>
-          <upward>0 0 1</upward>
-	  <cp>0.0 0.0 0.0</cp>
+          <aBdyXX>0.01125</aBdyXX>
+          <aBdyYY>0</aBdyYY>
+          <aBdyZZ>0</aBdyZZ>
+          <forward>1 0 0</forward>
+          <upward>0 0 1</upward>
+          <cp>-0.01 0 -0.025</cp>
           <wind name="wind">
             <topic>wind_base_link</topic>
@@ -417,9 +401,9 @@
     </plugin>
   </gazebo>
-  <!-- aft wing L&D plugin -->
+  <!-- airfoil plugins -->
   <gazebo>
     <plugin filename="librotors_gazebo_aerodynamics_plugin.so" name="aerodynamics_plugin">
       <robotNamespace>${namespace}</robotNamespace>
-      <aeroForcesVis>aero_force_vis_1</aeroForcesVis>
+      <aeroForcesVis>aero_force_vis_tail</aeroForcesVis>
       <airfoil>
         <segment name="EL">
@@ -431,5 +415,5 @@
           <seg_area>0.0112</seg_area>
           <seg_chord>0.08</seg_chord>
-          <aeroParamsYAML>${yaml_path}/---ic2_wing_airfoil.yaml</aeroParamsYAML>
+          <aeroParamsYAML>${yaml_path}/ic2_tail_airfoil.yaml</aeroParamsYAML>
           <wind name="wind">
             <topic>wind_base_link</topic>
@@ -444,5 +428,5 @@
           <seg_area>0.0112</seg_area>
           <seg_chord>0.08</seg_chord>
-          <aeroParamsYAML>${yaml_path}/---ic2_wing_airfoil.yaml</aeroParamsYAML>
+          <aeroParamsYAML>${yaml_path}/ic2_tail_airfoil.yaml</aeroParamsYAML>
           <wind name="wind">
             <topic>wind_base_link</topic>
@@ -457,5 +441,5 @@
           <seg_area>0.015</seg_area>
           <seg_chord>0.15</seg_chord>
-          <aeroParamsYAML>${yaml_path}/cl84b_tail_airfoil.yaml</aeroParamsYAML>
+          <aeroParamsYAML>${yaml_path}/ic2_tail_airfoil.yaml</aeroParamsYAML>
           <wind name="wind">
             <topic>wind_base_link</topic>
@@ -465,161 +449,160 @@
     </plugin>
   </gazebo>
-  <!-- front wing L&D plugin -->
   <gazebo>
-    <plugin filename="librotors_gazebo_aerodynamics_plugin.so" name="aerodynamics_plugin">
-      <robotNamespace>${namespace}</robotNamespace>
-      <aeroForcesVis>aero_force_vis_1</aeroForcesVis>
-      <airfoil>
-      <segment name="WL1">
-        <linkNameRef>${namespace}/wing_left</linkNameRef>
-        <linkNameAct>${namespace}/base_link</linkNameAct>
-        <forward>1 0 0</forward>
-        <upward>0 0 1</upward>
-        <cp>-0.05 0.0500 -0.005</cp>
-        <seg_area>0.020</seg_area>
-        <seg_chord>0.20</seg_chord>
-        <aeroParamsYAML>${yaml_path}/---ic2_wing_airfoil.yaml</aeroParamsYAML>
-        <wind name="wind">
-          <topic>wind_base_link</topic>
-        </wind>
-      </segment>
-      <segment name="WL2">
-        <linkNameRef>${namespace}/wing_left</linkNameRef>
-        <linkNameAct>${namespace}/base_link</linkNameAct>
-        <forward>1 0 0</forward>
-        <upward>0 0 1</upward>
-        <cp>-0.05 0.1625 -0.005</cp>
-        <seg_area>0.025</seg_area>
-        <seg_chord>0.20</seg_chord>
-        <aeroParamsYAML>${yaml_path}/---ic2_wing_airfoil.yaml</aeroParamsYAML>
-        <wind name="wind">
-          <topic>wind_base_link</topic>
-        </wind>
-        <indVel name="propeller_front_left">
-           <topic>propeller_front_left_slpstr</topic>
-        </indVel>
-      </segment>
-      <segment name="WL3">
-        <linkNameRef>${namespace}/wing_left</linkNameRef>
-        <linkNameAct>${namespace}/base_link</linkNameAct>
-        <forward>1 0 0</forward>
-        <upward>0 0 1</upward>
-        <cp>-0.05 0.2875 -0.005</cp>
-        <seg_area>0.025</seg_area>
-        <seg_chord>0.20</seg_chord>
-        <aeroParamsYAML>${yaml_path}/---ic2_wing_airfoil.yaml</aeroParamsYAML>
-        <control>
-          <cs name="aileron_left">
-              <controlJoint>${namespace}/aileron_left_joint</controlJoint>
-              <radToCLift>3</radToCLift> <!-- !!!!!!!!!!!!!!!!! -->
-              <radToCDrag>0.0</radToCDrag>
-              <radToCPitch>0.0</radToCPitch>
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