Commit message: New Back-up Icarus_2c should be working good enough, and Scintilla_01 is on its way to work

File: rotors_simulator/rotors_description/urdf/SCINTILLA_01.xacro (robot description, xacro)
@@ -23,21 +23,17 @@
   <xacro:property name="PI" value="3.1415926535897931" />
   <!-- Component masses -->
-  <xacro:property name="mass_aileron" value="0.01" /> <!-- [kg] 0.001-->
-  <xacro:property name="mass_elevator" value="0.05" /> <!-- [kg] 0.022-->
+  <xacro:property name="mass_aileron" value="0.068" /> <!-- [kg] -->
+  <xacro:property name="mass_elevator" value="0.304" /> <!-- [kg] -->
   <!-- Aileron properties -->
-  <xacro:property name="aileron_length" value="0.09" /> <!-- [m] 0.03-->
-  <xacro:property name="aileron_width" value="0.185" /> <!-- [m] 0.15-->
-  <xacro:property name="aileron_height" value="0.03" /> <!-- [m] 0.01-->
-  <!-- <xacro:property name="aileron_min_angle" value="-0.349066" />  [rad] -->
-  <!-- <xacro:property name="aileron_max_angle" value="0.349066" />  [rad]  -->
+  <xacro:property name="aileron_length" value="0.062" /> <!-- [m] -->
+  <xacro:property name="aileron_width" value="1.034" /> <!-- [m] -->
+  <xacro:property name="aileron_height" value="0.02" /> <!-- [m] -->
   <xacro:property name="aileron_color" value="Red" />
   <xacro:property name="aileron_left_mesh_file" value="package://rotors_description/meshes/techpod/techpod_aileron_left.dae" />
   <xacro:property name="aileron_right_mesh_file" value="package://rotors_description/meshes/techpod/techpod_aileron_right.dae" />
   <!-- Elevator properties -->
-  <xacro:property name="elevator_length" value="0.08" /> <!-- [m] -->
-  <xacro:property name="elevator_width" value="0.4" /> <!-- [m] -->
-  <xacro:property name="elevator_height" value="0.01" /> <!-- [m] 0.05-->
-  <!-- <xacro:property name="elevator_min_angle" value="-0.349066" /> [rad] -->
-  <!-- <xacro:property name="elevator_max_angle" value="0.349066" /> [rad] -->
+  <xacro:property name="elevator_length" value="0.1" /> <!-- [m] -->
+  <xacro:property name="elevator_width" value="0.8" /> <!-- [m] -->
+  <xacro:property name="elevator_height" value="0.01" /> <!-- [m] -->
   <xacro:property name="elevator_color" value="Blue" />
   <xacro:property name="elevator_mesh_file" value="package://rotors_description/meshes/techpod/techpod_elevator.dae" />
@@ -48,6 +44,5 @@
   <!-- Inertia of the elevator, assuming it is a cuboid -->
   <xacro:property name="elevator_inertia">
-    <xacro:box_inertia x="0.1" y="0.4" z="0.01" mass="${mass_elevator}"/> <!--Changed-->
-	<!-- <xacro:box_inertia x="${elevator_length}" y="${elevator_width}" z="${elevator_height}" mass="${mass_elevator}" />  -->
+	   <xacro:box_inertia x="${elevator_length}" y="${elevator_width}" z="${elevator_height}" mass="${mass_elevator}" />
   </xacro:property>
   <!-- Servo PD controller paramters, tune after inertias of actuated links are set -->
@@ -62,19 +57,21 @@
     <d>0.01</d>
   </xacro:property>
+  <xacro:property name="rud_srv_params">
+    <slew>5</slew>
+    <p>0.035</p>
+    <d>0.01</d>
+  </xacro:property>
   <xacro:property name="wing_srv_params">
     <slew>0.52</slew>
-    <p>5</p>
+    <p>20</p>
     <d>0</d>
   </xacro:property>
-  <xacro:property name="distance_origin_ground" value="0.0" />
-  <xacro:property name="ram_eff" value="0.5" />
-  <xacro:property name="slip_eff" value="0.5" />
   <xacro:include filename="$(find rotors_description)/urdf/fixed_wing_X_base.xacro" />
-  <!-- Fuselage -->
+  <!-- Fuselage - Ineritas and Masses need to be checked -->
   <link name="${namespace}/base_link">
       <inertial>
-        <mass value="0.6" /> <!--changed from 0.8 -->
-        <inertia ixx="0.0035" ixy="0.0" ixz="0.01" iyy="0.0082" iyz="0.0" izz="0.0045" />
-        <origin xyz="${distance_origin_ground} 0 0" rpy="0 0 0" />
+        <mass value="6.64" />
+        <inertia ixx="0.044958" ixy="0.002614" ixz="0.019172" iyy="0.254345" iyz="0.000036" izz="0.233503" />
+        <origin xyz="-0.2775 0 0" rpy="0 0 0" />
       </inertial>
       <visual>
@@ -85,46 +82,12 @@
       </visual>
       <collision>
-        <origin xyz="0.1 -0.1 -0.1" rpy="0 0 0" />
+        <origin xyz="-0.3 0 0" rpy="0 0 0" />
         <geometry>
-          <sphere radius="0.05" />
+          <box size="0.5 0.2 0.2" />
         </geometry>
       </collision>
-      <collision>
-        <origin xyz="0.1 0.1 -0.1" rpy="0 0 0" />
-        <geometry>
-          <sphere radius="0.05" />
-        </geometry>
-      </collision>
-      <collision>
-        <origin xyz="-0.4 0 -0.1" rpy="0 0 0" />
-        <geometry>
-          <sphere radius="0.05" />
-        </geometry>
-      </collision>
   </link>
   <gazebo reference="${namespace}/base_link">
     <material>Gazebo/White</material>
-  </gazebo>
-<!-- Center of Gravity manipulation -->
-  <joint name="${namespace}/CG_joint" type="fixed">
-    <parent link="${namespace}/base_link" />
-    <child link="${namespace}/CG" />
-    <origin xyz="-0.025 0 -0.05" rpy="0 0 0" />
-  </joint>
-  <link name="${namespace}/CG">
-    <inertial>
-      <mass value="0.2" />
-      <inertia ixx="0.0035" ixy="0.0" ixz="0.01" iyy="0.0082" iyz="0.0" izz="0.0045" />
-      <origin xyz="0 0 0" rpy="0 0 0" />
-    </inertial>
-    <visual>
-      <origin xyz="0 0 0" rpy="0 0 0" />
-      <geometry>
-        <cylinder radius="0.025" length="0.02" />
-      </geometry>
-    </visual>
-  </link>
-  <gazebo reference="${namespace}/CG">
-    <material>Gazebo/Black</material>
   </gazebo>
   <!-- Wing -->
@@ -132,5 +95,5 @@
     <parent link="${namespace}/base_link" />
     <child link="${namespace}/wing_left" />
-    <origin xyz="-0.35 0.12 0.11" rpy="0 0 0" />
+    <origin xyz="-0.377 0.12 0.114" rpy="0 0 0" />
     <axis xyz="0 1 0" />
     <limit upper="0.0" lower="-1.57" effort="10" velocity="20"/>
@@ -139,12 +102,10 @@
   <link name="${namespace}/wing_left">
     <inertial>
-      <mass value="0.1" />
-      <!--<inertia ixx="0.01" ixy="0.0" ixz="0.01" iyy="0.0" iyz="0.0" izz="0.01" />
-      <origin xyz="0 -0.060 0" rpy="0 0 0" /> -->
-      <inertia ixx="0.0273" ixy="0.0" ixz="0.0002" iyy="0.0009" iyz="0.0" izz="0.0278"/>
-      <origin xyz="0 0 0" rpy="0 0 0" />
-    </inertial>
-    <visual>
-      <origin xyz="0.345 -0.125 -0.11" rpy="0 0 ${pi/2}" />
+      <mass value="0.248" />
+      <inertia ixx="0.034569" ixy="0.000234" ixz="0.000089" iyy="0.001145" iyz="0.000017" izz="0.035653" />
+      <origin xyz="0 0.519 0" rpy="0 0 0" />
+    </inertial>
+    <visual>
+      <origin xyz="0.372 -0.125 -0.114" rpy="0 0 ${pi/2}" />
       <geometry>
         <mesh filename="package://rotors_description/meshes/IGNIS/SCINTILLA/Wings.stl" scale="0.001 0.001 0.001" />
@@ -152,7 +113,7 @@
     </visual>
     <collision>
-        <origin xyz="-0.05 0.25 0" rpy="0 0 0" />
+        <origin xyz="-0.05 0.52 0" rpy="0 0 0" />
         <geometry>
-          <box size="0.1 0.35 0.01" />
+          <box size="0.1 1.0 0.01" />
         </geometry>
     </collision>
@@ -164,5 +125,5 @@
     <parent link="${namespace}/base_link" />
     <child link="${namespace}/wing_right" />
-    <origin xyz="-0.35 -0.12 0.11" rpy="0 0 0" />
+    <origin xyz="-0.377 -0.12 0.114" rpy="0 0 0" />
     <axis xyz="0 1 0" />
     <limit upper="0.0" lower="-1.57" effort="10" velocity="20"/>
@@ -170,13 +131,11 @@
   </joint>
   <link name="${namespace}/wing_right">
-      <inertial>
-        <mass value="0.1" />
-        <!-- <inertia ixx="0.01" ixy="0.0" ixz="0.01" iyy="0.0" iyz="0.0" izz="0.01" />
-        <origin xyz="0 0.060 0" rpy="0 0 0" /> -->
-        <inertia ixx="0.0273" ixy="0.0" ixz="0.0002" iyy="0.0009" iyz="0.0" izz="0.0278" />
-        <origin xyz="0 0 0" rpy="0 0 0" />
-      </inertial>
+    <inertial>
+      <mass value="0.248" />
+      <inertia ixx="0.034569" ixy="0.000234" ixz="0.000089" iyy="0.001145" iyz="0.000017" izz="0.035653" />
+      <origin xyz="0 -0.519 0" rpy="0 0 0" />
+    </inertial>
       <visual>
-        <origin xyz="0.345 -1.155 -0.11" rpy="0 0 ${pi/2}" />
+        <origin xyz="0.372 -1.155 -0.114" rpy="0 0 ${pi/2}" />
         <geometry>
           <mesh filename="package://rotors_description/meshes/IGNIS/SCINTILLA/Wings.stl" scale="0.001 0.001 0.001" />
@@ -184,7 +143,7 @@
       </visual>
       <collision>
-        <origin xyz="-0.05 -0.25 0" rpy="0 0 0" />
+        <origin xyz="-0.05 -0.52 0" rpy="0 0 0" />
         <geometry>
-          <box size="0.1 0.35 0.01" />
+          <box size="0.1 1.0 0.01" />
         </geometry>
     </collision>
@@ -195,5 +154,5 @@
   <!-- Ailerons -->
   <joint name="${namespace}/aileron_left_joint" type="revolute">
-    <origin xyz="-0.08 0.505 -0.02" rpy="0 0 0" />
+    <origin xyz="-0.08 0.519 -0.02" rpy="0 0 0" />
     <axis xyz="0 -1 0" />
     <parent link="${namespace}/wing_left" />
@@ -207,5 +166,5 @@
     </inertial>
     <visual>
-      <origin xyz="0.428 -0.62 -0.09" rpy="0 0 ${pi/2}" />
+      <origin xyz="0.455 -0.644 -0.09" rpy="0 0 ${pi/2}" />
       <geometry>
           <mesh filename="package://rotors_description/meshes/IGNIS/SCINTILLA/Aileron.stl" scale="0.001 0.001 0.001" />
@@ -217,5 +176,5 @@
   </gazebo>
   <joint name="${namespace}/aileron_right_joint" type="revolute">
-    <origin xyz="-0.08 -0.415 -0.02" rpy="0 0 0" />
+    <origin xyz="-0.08 -0.519 -0.02" rpy="0 0 0" />
     <axis xyz="0 -1 0" />
     <parent link="${namespace}/wing_right" />
@@ -229,5 +188,5 @@
     </inertial>
     <visual>
-      <origin xyz="0.428 -0.745 -0.09" rpy="0 0 ${pi/2}" />
+      <origin xyz="0.455 -0.636 -0.09" rpy="0 0 ${pi/2}" />
       <geometry>
           <mesh filename="package://rotors_description/meshes/IGNIS/SCINTILLA/Aileron.stl" scale="0.001 0.001 0.001" />
@@ -238,5 +197,5 @@
     <material>Gazebo/${aileron_color}</material>
   </gazebo>
-<!-- Vertical Stabilizer -->
+<!-- Tail -->
   <joint name="${namespace}/tail_joint" type="fixed">
     <parent link="${namespace}/base_link" />
@@ -246,7 +205,7 @@
   <link name="${namespace}/tail">
     <inertial>
-      <mass value="0.2" />
-      <inertia ixx="0.0035" ixy="0.0" ixz="0.01" iyy="0.0082" iyz="0.0" izz="0.0045" />
-      <origin xyz="0 0 0" rpy="0 0 0" />
+      <mass value="0.29" />
+      <inertia ixx="0.019969" ixy="0.0" ixz="0.000967" iyy="0.005362" iyz="0.0" izz="0.023453" />
+      <origin xyz="-0.13 0 0" rpy="0 0 0" />
     </inertial>
     <visual>
@@ -259,4 +218,28 @@
   <gazebo reference="${namespace}/CG">
     <material>Gazebo/Black</material>
+  </gazebo>
+  <!-- Rudder -->
+  <joint name="${namespace}/rudder_joint" type="revolute">
+    <origin xyz="-0.15 0 0.0" rpy="0 0 0" />
+    <axis xyz="0 0 1" />
+    <parent link="${namespace}/tail" />
+    <child link="${namespace}/rudder" />
+    <limit upper="0.53" lower="-0.53" effort="10" velocity="20"/>
+  </joint>
+  <link name="${namespace}/rudder">
+    <inertial>
+      <mass value="0.024" />
+      <xacro:box_inertia x="0.06" y="0.01" z="0.15" mass="0.024" />
+      <origin xyz="0 0 0.08" rpy="0 0 0" />
+    </inertial>
+    <visual>
+      <origin xyz="1.225 0.0 0.0" rpy="0 0 ${pi/2}" />
+      <geometry>
+          <mesh filename="package://rotors_description/meshes/IGNIS/SCINTILLA/Rudder.stl" scale="0.001 0.001 0.001" />
+      </geometry>
+    </visual>
+  </link>
+  <gazebo reference="${namespace}/aileron_left">
+    <material>Gazebo/${aileron_color}</material>
   </gazebo>
   <!-- Elevator -->
@@ -284,6 +267,33 @@
   </gazebo>
   <!-- Propellers -->
+  <joint name="${namespace}/propeller_front_left_left_joint" type="continuous">
+    <origin xyz="0.087 0.778 0" rpy="0 ${0.5*pi} 0" />
+    <axis xyz="0 0 1" />
+    <parent link="${namespace}/wing_left" />
+    <child link="${namespace}/propeller_front_left_left" />
+  </joint>
+  <link name="${namespace}/propeller_front_left_left">
+    <inertial>
+      <mass value="0.017" />
+      <xacro:cylinder_inertia r="0.14" h="0.02" mass="0.017" />
+    </inertial>
+    <visual>
+      <origin xyz="0 0 0" rpy="0 0 0" />
+      <geometry>
+        <mesh filename="package://rotors_description/meshes/tiltwing/iris_prop_ccw.dae" scale="0.9 0.9 0.9"/>
+      </geometry>
+    </visual>
+    <visual>
+      <origin xyz="0 0 -0.015" rpy="0 0 0" />
+      <geometry>
+        <cylinder radius="0.025" length="0.02" />
+      </geometry>
+    </visual>
+  </link>
+  <gazebo reference="${namespace}/propeller_front_left_left">
+    <material>Gazebo/DarkGrey</material>
+  </gazebo>
   <joint name="${namespace}/propeller_front_left_joint" type="continuous">
-    <origin xyz="0.03 0.225 0" rpy="0 ${0.5*pi} 0" />
+    <origin xyz="0.087 0.261 0" rpy="0 ${0.5*pi} 0" />
     <axis xyz="0 0 1" />
     <parent link="${namespace}/wing_left" />
@@ -292,6 +302,6 @@
   <link name="${namespace}/propeller_front_left">
     <inertial>
-      <mass value="0.0125" />
-      <xacro:cylinder_inertia r="0.14" h="0.02" mass="0.0125" />
+      <mass value="0.017" />
+      <xacro:cylinder_inertia r="0.14" h="0.02" mass="0.017" />
     </inertial>
     <visual>
@@ -312,5 +322,5 @@
   </gazebo>
   <joint name="${namespace}/propeller_front_right_joint" type="continuous">
-    <origin xyz="0.03 -0.225 0" rpy="0 ${0.5*pi} 0" />
+    <origin xyz="0.087 -0.261 0" rpy="0 ${0.5*pi} 0" />
     <axis xyz="0 0 1" />
     <parent link="${namespace}/wing_right" />
@@ -319,6 +329,6 @@
   <link name="${namespace}/propeller_front_right">
     <inertial>
-      <mass value="0.0125" />
-      <xacro:cylinder_inertia r="0.14" h="0.02" mass="0.0125" />
+      <mass value="0.017" />
+      <xacro:cylinder_inertia r="0.14" h="0.02" mass="0.017" />
     </inertial>
     <visual>
@@ -338,6 +348,33 @@
     <material>Gazebo/DarkGrey</material>
   </gazebo>
+  <joint name="${namespace}/propeller_front_right_right_joint" type="continuous">
+    <origin xyz="0.087 -0.778 0" rpy="0 ${0.5*pi} 0" />
+    <axis xyz="0 0 1" />
+    <parent link="${namespace}/wing_right" />
+    <child link="${namespace}/propeller_front_right_right" />
+  </joint>
+  <link name="${namespace}/propeller_front_right_right">
+    <inertial>
+      <mass value="0.017" />
+      <xacro:cylinder_inertia r="0.14" h="0.02" mass="0.017" />
+    </inertial>
+    <visual>
+      <origin xyz="0 0 0" rpy="0 0 0" />
+      <geometry>
+        <mesh filename="package://rotors_description/meshes/tiltwing/iris_prop_ccw.dae" scale="0.9 0.9 0.9"/>
+      </geometry>
+    </visual>
+    <visual>
+      <origin xyz="0 0 -0.015" rpy="0 0 0" />
+      <geometry>
+        <cylinder radius="0.025" length="0.02" />
+      </geometry>
+    </visual>
+  </link>
+  <gazebo reference="${namespace}/propeller_front_right_right">
+    <material>Gazebo/DarkGrey</material>
+  </gazebo>
   <joint name="${namespace}/propeller_back_joint" type="continuous">
-    <origin xyz="-0.53 0 0" rpy="0 0 0" />
+    <origin xyz="-1.39 0 0.02" rpy="0 0 0" />
     <axis xyz="0 0 1" />
     <parent link="${namespace}/base_link" />
@@ -346,6 +383,6 @@
   <link name="${namespace}/propeller_back">
     <inertial>
-      <mass value="0.1" /> <!-- 0.01 -->
-      <xacro:cylinder_inertia r="0.08" h="0.01" mass="0.01" />
+      <mass value="0.122" />
+      <xacro:cylinder_inertia r="0.08" h="0.01" mass="0.122" />
     </inertial>
     <visual>
@@ -356,5 +393,5 @@
     </visual>
     <visual>
-      <origin xyz="0 0 -0.01" rpy="0 0 0" />
+      <origin xyz="0 0 -0.005" rpy="0 0 0" />
       <geometry>
         <cylinder radius="0.01" length="0.01" />
@@ -365,50 +402,37 @@
     <material>Gazebo/Orange</material>
   </gazebo>
-  <!--
-  <joint name="${namespace}/propeller_back_right_joint" type="continuous">
-    <origin xyz="0.0 -0.185 0" rpy="0 ${0.5*pi} 0" />
-    <axis xyz="0 0 1" />
-    <parent link="${namespace}/elevator" />
-    <child link="${namespace}/propeller_back_right" />
-  </joint>
-  <link name="${namespace}/propeller_back_right">
-    <inertial>
-      <mass value="0.01" />
-      <xacro:cylinder_inertia r="0.08" h="0.01" mass="0.01" />
-    </inertial>
-    <visual>
-      <origin xyz="0 0 0.04" rpy="0 0 0" />
-      <geometry>
-        <mesh filename="package://rotors_description/meshes/IGNIS/ICARUS_2/iris_prop_ccw.dae" scale="0.6 0.6 0.6"/>
-      </geometry>
-    </visual>
-    <visual>
-      <origin xyz="0 0 0.03" rpy="0 0 0" />
-      <geometry>
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
Commit message: Scintilla is flying pretty well

File: rotors_simulator/rotors_description/urdf/ICARUS_2c.xacro (robot description, xacro)
@@ -66,5 +66,5 @@
   <link name="${namespace}/base_link">
       <inertial>
-        <origin xyz="-0.01 0 -0.025" rpy="0 0 0" /> <!-- CG has to be in these coordinates -->
+        <origin xyz="0.048 0 -0.025" rpy="0 0 0" /> <!-- With the current weights it should be 0.048 0 -0.025 -->
         <mass value="1.0" />
         <inertia ixx="0.0033" ixy="0.0" ixz="0.0" iyy="0.0473" iyz="0.0" izz="0.0472" />
@@ -297,5 +297,5 @@
   </gazebo>
   <joint name="${namespace}/propeller_back_joint" type="continuous">
-    <origin xyz="-0.53 0 0" rpy="0 0 0" />
+    <origin xyz="-0.43 0 0" rpy="0 0 0" />
     <axis xyz="0 0 1" />
     <parent link="${namespace}/base_link" />
@@ -305,5 +305,5 @@
     <inertial>
       <mass value="0.1" />
-      <xacro:cylinder_inertia r="0.08" h="0.01" mass="0.01" />
+      <xacro:cylinder_inertia r="0.08" h="0.01" mass="0.1" />
     </inertial>
     <visual>
@@ -330,5 +330,5 @@
         <linkNameRef>${namespace}/wing_left</linkNameRef>
         <linkNameAct>${namespace}/base_link</linkNameAct>
-        <cp>0.08 0.225 0</cp>			<!-- !!! -->
+        <cp>0.08 0.225 0</cp>
         <axisPosRot>-1 0 0</axisPosRot>
         <turnDir>cw</turnDir>

File: rotors_simulator/rotors_description/urdf/SCINTILLA_01.xacro (robot description, xacro)
@@ -73,5 +73,5 @@
         <mass value="6.64" />
         <inertia ixx="0.044958" ixy="0.002614" ixz="0.019172" iyy="0.254345" iyz="0.000036" izz="0.233503" />
-        <origin xyz="-0.2775 0 0" rpy="0 0 0" />
+        <origin xyz="-0.37 0 0" rpy="0 0 0" /> <!-- -0.33 -->
       </inertial>
       <visual>
@@ -878,5 +878,5 @@
         </channel>
         <channel name="propeller_front_right_right">
-          <input_index>3</input_index>
+          <input_index>4</input_index>
           <input_offset>1</input_offset>
           <input_scaling>316</input_scaling>
@@ -887,5 +887,5 @@
         </channel>
         <channel name="propeller_front_right_right_anim">
-           <input_index>3</input_index>
+           <input_index>4</input_index>
            <input_offset>1</input_offset>
            <input_scaling>20</input_scaling>
@@ -896,5 +896,5 @@
         </channel>
         <channel name="propeller_back">
-          <input_index>4</input_index>
+          <input_index>5</input_index>
           <input_offset>1</input_offset>
           <input_scaling>607</input_scaling>
@@ -905,5 +905,5 @@
         </channel>
         <channel name="propeller_back_anim">
-           <input_index>4</input_index>
+           <input_index>5</input_index>
            <input_offset>1</input_offset>
            <input_scaling>20</input_scaling>
@@ -914,5 +914,5 @@
         </channel>
         <channel name="wing_left">
-           <input_index>5</input_index>
+           <input_index>8</input_index>
            <input_offset>0</input_offset>
            <input_scaling>-1.57</input_scaling>
@@ -926,5 +926,5 @@
         </channel>
         <channel name="wing_right">
-           <input_index>5</input_index>
+           <input_index>8</input_index>
            <input_offset>0</input_offset>
            <input_scaling>-1.57</input_scaling>
@@ -938,5 +938,5 @@
         </channel>
         <channel name="aileron_left">
-          <input_index>6</input_index>
+          <input_index>9</input_index>
           <input_offset>0</input_offset>
           <input_scaling>0.53</input_scaling>
@@ -951,5 +951,5 @@
         </channel>
         <channel name="aileron_right">
-          <input_index>7</input_index>
+          <input_index>10</input_index>
           <input_offset>0</input_offset>
           <input_scaling>-0.53</input_scaling>
@@ -964,5 +964,5 @@
         </channel>
         <channel name="elevator">
-          <input_index>8</input_index>
+          <input_index>11</input_index>
           <input_offset>0</input_offset>
           <input_scaling>-1.57</input_scaling>
@@ -976,5 +976,5 @@
         </channel>
         <channel name="rudder">
-          <input_index>9</input_index>
+          <input_index>12</input_index>
           <input_offset>0</input_offset>
           <input_scaling>-0.53</input_scaling>

File: rotors_simulator/rotors_description/urdf/aeromini_base.xacro (robot description, xacro)
@@ -1,5 +1,5 @@
 <?xml version="1.0"?>
 <!--
-  Copyright 2019 David Rohr, ASL, ETH Zurich, Switzerland
+  Copyright 2021 David Rohr, ASL, ETH Zurich, Switzerland
   Licensed under the Apache License, Version 2.0 (the "License");
   you may not use this file except in compliance with the License.
@@ -12,18 +12,13 @@
   limitations under the License.
 -->
-<robot name="SCINTILLA_01" xmlns:xacro="http://ros.org/wiki/xacro">
+<robot name="aeromini" xmlns:xacro="http://ros.org/wiki/xacro">
   <xacro:include filename="$(find rotors_description)/urdf/component_snippets.xacro" />
   <!-- Instantiate fixed wing "mechanics" -->
-  <xacro:include filename="$(find rotors_description)/urdf/SCINTILLA_01.xacro" />
+  <xacro:include filename="$(find rotors_description)/urdf/aeromini.xacro" />
   <!-- Mount an ADIS16448 IMU. -->
   <xacro:default_imu namespace="${namespace}" parent_link="${namespace}/base_link" >
-    <origin xyz="-0.45 0 0.065" rpy="0 0 0" />  <!-- !!! Where our Pixhawk lies-->
+    <origin xyz="0.14 -0.01 0.07" rpy="0 0 0" />
   </xacro:default_imu>
   <!-- Mount a GPS.-->
-  <!--<xacro:default_gps
-    namespace="${namespace}"
-    parent_link="${namespace}/base_link">
-    <origin xyz="0 0 0" rpy="0 0 0" />
-  </xacro:default_gps>-->
   <xacro:gps_plugin_macro
     namespace="${namespace}"
@@ -39,5 +34,5 @@
     enable_delay = "false">
     <xacro:cube_inertia l="0.02" mass="0.015" />
-    <origin xyz="-0.417 0 0" rpy="0 0 0" />
+    <origin xyz="0 0 0" rpy="0 0 0" />
   </xacro:gps_plugin_macro>
   <xacro:gps_plugin_macro
@@ -54,6 +49,13 @@
     enable_delay = "false">
     <xacro:cube_inertia l="0.02" mass="0.001" />
-    <origin xyz="-0.417 0 0" rpy="0 0 0" />
+    <origin xyz="0 0 0" rpy="0 0 0" />
   </xacro:gps_plugin_macro>
+  <xacro:default_camera
+    namespace="${namespace}"
+    parent_link="${namespace}/base_link"
+    camera_suffix="cam_front">
+    <origin xyz="-0.2 0.10 0.0" rpy="0 0 1.4" />
+  </xacro:default_camera>
+  <!--
   <xacro:camera_macro_2
     namespace="${namespace}"
@@ -73,5 +75,5 @@
     <mesh filename="package://rotors_description/meshes/vi_camera.dae" scale="1 1 1" />
     <xacro:cube_inertia l="0.02" mass="0.01" />
-    <origin xyz="-0.417 0 0" rpy="0 0.2 0" />
-  </xacro:camera_macro_2>
+    <origin xyz="-2 0 0.5" rpy="0 0.2 0" />
+  </xacro:camera_macro_2>-->
 </robot>
