Commit message: Elevator tilt limitations corrected

File: rotors_simulator/rotors_description/urdf/ICARUS_2c.xacro (robot description, xacro)
@@ -49,6 +49,6 @@
   <xacro:property name="ail_srv_params">
     <slew>5</slew>
-    <p>0.0004</p>
-    <d>0.00002</d>
+    <p>0.00004</p>
+    <d>0.002</d>
   </xacro:property>
   <xacro:property name="elev_srv_params">
@@ -221,5 +221,5 @@
     <parent link="${namespace}/base_link" />
     <child link="${namespace}/elevator" />
-    <limit upper="0.3" lower="-1.57" effort="50" velocity="50"/>
+    <limit upper="0.53" lower="-0.53" effort="50" velocity="50"/>
   </joint>
   <link name="${namespace}/elevator">
@@ -719,5 +719,5 @@
           <input_index>6</input_index>
           <input_offset>0</input_offset>
-          <input_scaling>-1.57</input_scaling>
+          <input_scaling>-0.53</input_scaling>
           <zero_position_disarmed>0</zero_position_disarmed>
           <zero_position_armed>0</zero_position_armed>

File: rotors_simulator/rotors_description/urdf/SCINTILLA_01.xacro (robot description, xacro)
@@ -30,6 +30,4 @@
   <xacro:property name="aileron_height" value="0.02" /> <!-- [m] -->
   <xacro:property name="aileron_color" value="Red" />
-  <xacro:property name="aileron_left_mesh_file" value="package://rotors_description/meshes/techpod/techpod_aileron_left.dae" />
-  <xacro:property name="aileron_right_mesh_file" value="package://rotors_description/meshes/techpod/techpod_aileron_right.dae" />
   <!-- Elevator properties -->
   <xacro:property name="elevator_length" value="0.1" /> <!-- [m] -->
@@ -49,16 +47,16 @@
   <xacro:property name="ail_srv_params">
     <slew>5</slew>
-    <p>0.0004</p>
-    <d>0.00002</d>
+    <p>0.00004</p>
+    <d>0.002</d>
   </xacro:property>
   <xacro:property name="elev_srv_params">
     <slew>4</slew>
-    <p>0.035</p>
-    <d>0.01</d>
+    <p>0.09</p>
+    <d>0.009</d>
   </xacro:property>
   <xacro:property name="rud_srv_params">
     <slew>5</slew>
-    <p>0.035</p>
-    <d>0.01</d>
+    <p>0.00004</p>
+    <d>0.002</d>
   </xacro:property>
   <xacro:property name="wing_srv_params">
@@ -240,5 +238,5 @@
     </visual>
   </link>
-  <gazebo reference="${namespace}/aileron_left">
+  <gazebo reference="${namespace}/rudder">
     <material>Gazebo/${aileron_color}</material>
   </gazebo>
@@ -249,5 +247,5 @@
     <parent link="${namespace}/base_link" />
     <child link="${namespace}/elevator" />
-    <limit upper="0.3" lower="-1.57" effort="50" velocity="50"/>
+    <limit upper="0.53" lower="-0.53" effort="50" velocity="50"/>
   </joint>
   <link name="${namespace}/elevator">
@@ -915,6 +913,6 @@
         <channel name="wing_left">
            <input_index>8</input_index>
-           <input_offset>0</input_offset>
-           <input_scaling>-1.57</input_scaling>
+           <input_offset>1</input_offset>
+           <input_scaling>-${1.57*0.5}</input_scaling>
            <zero_position_disarmed>0</zero_position_disarmed>
            <zero_position_armed>0</zero_position_armed>
@@ -927,6 +925,6 @@
         <channel name="wing_right">
            <input_index>8</input_index>
-           <input_offset>0</input_offset>
-           <input_scaling>-1.57</input_scaling>
+           <input_offset>1</input_offset>
+           <input_scaling>-${1.57*0.5}</input_scaling>
            <zero_position_disarmed>0</zero_position_disarmed>
            <zero_position_armed>0</zero_position_armed>
@@ -939,4 +937,17 @@
         <channel name="aileron_left">
           <input_index>9</input_index>
+          <input_offset>0</input_offset>
+          <input_scaling>-0.53</input_scaling>
+          <zero_position_disarmed>0</zero_position_disarmed>
+          <zero_position_armed>0</zero_position_armed>
+          <joint_control_type>servo</joint_control_type>
+          <servo_params>
+            <xacro:insert_block name="ail_srv_params" />
+          </servo_params>
+          <joint_name>${namespace}/aileron_left_joint</joint_name>
+          <gztopic>aileron_left_pos</gztopic>
+        </channel>
+        <channel name="aileron_right">
+          <input_index>10</input_index>
           <input_offset>0</input_offset>
           <input_scaling>0.53</input_scaling>
@@ -947,17 +958,4 @@
             <xacro:insert_block name="ail_srv_params" />
           </servo_params>
-          <joint_name>${namespace}/aileron_left_joint</joint_name>
-          <gztopic>aileron_left_pos</gztopic>
-        </channel>
-        <channel name="aileron_right">
-          <input_index>10</input_index>
-          <input_offset>0</input_offset>
-          <input_scaling>-0.53</input_scaling>
-          <zero_position_disarmed>0</zero_position_disarmed>
-          <zero_position_armed>0</zero_position_armed>
-          <joint_control_type>servo</joint_control_type>
-          <servo_params>
-            <xacro:insert_block name="ail_srv_params" />
-          </servo_params>
           <joint_name>${namespace}/aileron_right_joint</joint_name>
           <gztopic>aileron_right_pos</gztopic>
@@ -966,5 +964,5 @@
           <input_index>11</input_index>
           <input_offset>0</input_offset>
-          <input_scaling>-1.57</input_scaling>
+          <input_scaling>-0.53</input_scaling>
           <zero_position_disarmed>0</zero_position_disarmed>
           <zero_position_armed>0</zero_position_armed>
@@ -985,6 +983,6 @@
             <xacro:insert_block name="rud_srv_params" />
           </servo_params>
-          <joint_name>${namespace}/aileron_right_joint</joint_name>
-          <gztopic>aileron_right_pos</gztopic>
+          <joint_name>${namespace}/rudder_joint</joint_name>
+          <gztopic>rudder_pos</gztopic>
         </channel>
       </control_channels>

Commit message: Scintilla should be ready?

File: rotors_simulator/rotors_description/urdf/ICARUS_2c.xacro (robot description, xacro)
@@ -66,5 +66,5 @@
   <link name="${namespace}/base_link">
       <inertial>
-        <origin xyz="0.048 0 -0.025" rpy="0 0 0" /> <!-- With the current weights it should be 0.048 0 -0.025 -->
+        <origin xyz="0.05 0 -0.037" rpy="0 0 0" /> <!-- With the current weights it should be 0.0468 0 -0.037 -->
         <mass value="1.0" />
         <inertia ixx="0.0033" ixy="0.0" ixz="0.0" iyy="0.0473" iyz="0.0" izz="0.0472" />
@@ -217,5 +217,5 @@
   <!-- Elevator -->
   <joint name="${namespace}/elevator_joint" type="revolute">
-    <origin xyz="-0.465 0 0.0" rpy="0 0 0" />
+    <origin xyz="-0.40 0 0.0" rpy="0 0 0" />
     <axis xyz="0 -1 0" />
     <parent link="${namespace}/base_link" />
@@ -297,5 +297,5 @@
   </gazebo>
   <joint name="${namespace}/propeller_back_joint" type="continuous">
-    <origin xyz="-0.43 0 0" rpy="0 0 0" />
+    <origin xyz="-0.445 0 0" rpy="0 0 0" />
     <axis xyz="0 0 1" />
     <parent link="${namespace}/base_link" />
@@ -364,5 +364,5 @@
         <linkNameRef>${namespace}/base_link</linkNameRef>
         <linkNameAct>${namespace}/base_link</linkNameAct>
-        <cp>-0.53 0 0</cp>
+        <cp>-0.445 0 0</cp>
         <axisPosRot>0 0 1</axisPosRot>
         <turnDir>ccw</turnDir>
@@ -412,5 +412,5 @@
           <forward>1 0 0</forward>
           <upward>0 0 1</upward>
-          <cp>-0.03 0.1 0.0</cp>
+          <cp>0.0 0.1 0.0</cp>
           <seg_area>0.0112</seg_area>
           <seg_chord>0.08</seg_chord>
@@ -425,5 +425,5 @@
           <forward>1 0 0</forward>
           <upward>0 0 1</upward>
-          <cp>-0.03 -0.1 0.0</cp>
+          <cp>0.0 -0.1 0.0</cp>
           <seg_area>0.0112</seg_area>
           <seg_chord>0.08</seg_chord>
@@ -438,5 +438,5 @@
           <forward>1 0 0</forward>
           <upward>0 1 0</upward>
-          <cp>-0.41 0 0.1</cp>
+          <cp>-0.38 0 0.1</cp>
           <seg_area>0.015</seg_area>
           <seg_chord>0.15</seg_chord>
@@ -459,5 +459,5 @@
           <forward>1 0 0</forward>
           <upward>0 0 1</upward>
-          <cp>0 0.0500 -0.005</cp>
+          <cp>0.0167 0.0500 -0.005</cp>
           <seg_area>0.020</seg_area>
           <seg_chord>0.20</seg_chord>
@@ -472,5 +472,5 @@
           <forward>1 0 0</forward>
           <upward>0 0 1</upward>
-          <cp>0 0.1625 -0.005</cp>
+          <cp>0.0167 0.1625 -0.005</cp>
           <seg_area>0.025</seg_area>
           <seg_chord>0.20</seg_chord>
@@ -488,5 +488,5 @@
           <forward>1 0 0</forward>
           <upward>0 0 1</upward>
-          <cp>0 0.2875 -0.005</cp>
+          <cp>0.0167 0.2875 -0.005</cp>
           <seg_area>0.025</seg_area>
           <seg_chord>0.20</seg_chord>
@@ -512,5 +512,5 @@
           <forward>1 0 0</forward>
           <upward>0 0 1</upward>
-          <cp>0 0.3950 -0.005</cp>
+          <cp>0.0167 0.3950 -0.005</cp>
           <seg_area>0.018</seg_area>
           <seg_chord>0.20</seg_chord>
@@ -533,5 +533,5 @@
           <forward>1 0 0</forward>
           <upward>0 0 1</upward>
-          <cp>0 -0.0500 -0.005</cp>
+          <cp>0.0167 -0.0500 -0.005</cp>
           <seg_area>0.020</seg_area>
           <seg_chord>0.20</seg_chord>
@@ -546,5 +546,5 @@
           <forward>1 0 0</forward>
           <upward>0 0 1</upward>
-          <cp>0 -0.1625 -0.005</cp>
+          <cp>0.0167 -0.1625 -0.005</cp>
           <seg_area>0.025</seg_area>
           <seg_chord>0.20</seg_chord>
@@ -562,5 +562,5 @@
           <forward>1 0 0</forward>
           <upward>0 0 1</upward>
-          <cp>0 -0.2875 -0.005</cp>
+          <cp>0.0167 -0.2875 -0.005</cp>
           <seg_area>0.025</seg_area>
           <seg_chord>0.20</seg_chord>
@@ -586,5 +586,5 @@
           <forward>1 0 0</forward>
           <upward>0 0 1</upward>
-          <cp>0 -0.3950 -0.005</cp>
+          <cp>0.0167 -0.3950 -0.005</cp>
           <seg_area>0.018</seg_area>
           <seg_chord>0.20</seg_chord>
@@ -630,6 +630,6 @@
       <actuatorsPubTopic>/command/motor_speed</actuatorsPubTopic>
       <linkName>${namespace}/base_link</linkName> <!-- reference link frame for airspeed and baro alt-->
-      <pitotPos>0 0 0</pitotPos>           <!-- pitot position wrt reference link -->
-      <baroPos>0 0 0</baroPos>            <!-- baro position wrt reference link -->
+      <pitotPos>-0.01 0 -0.025</pitotPos>           <!-- pitot position wrt reference link -->
+      <baroPos>-0.01 0 -0.025</baroPos>            <!-- baro position wrt reference link -->
       <wind name="wind">                          <!-- include wind in airspeed measurement -->
         <topic>wind_base_link</topic>
@@ -693,5 +693,5 @@
           <input_index>4</input_index>
           <input_offset>0</input_offset>
-          <input_scaling>0.53</input_scaling>
+          <input_scaling>-0.53</input_scaling>
           <zero_position_disarmed>0</zero_position_disarmed>
           <zero_position_armed>0</zero_position_armed>
@@ -706,5 +706,5 @@
           <input_index>5</input_index>
           <input_offset>0</input_offset>
-          <input_scaling>-0.53</input_scaling>
+          <input_scaling>0.53</input_scaling>
           <zero_position_disarmed>0</zero_position_disarmed>
           <zero_position_armed>0</zero_position_armed>
@@ -719,5 +719,5 @@
           <input_index>6</input_index>
           <input_offset>0</input_offset>
-          <input_scaling>-0.53</input_scaling>
+          <input_scaling>0.53</input_scaling>
           <zero_position_disarmed>0</zero_position_disarmed>
           <zero_position_armed>0</zero_position_armed>

File: rotors_simulator/rotors_description/urdf/SCINTILLA_01.xacro (robot description, xacro)
@@ -69,7 +69,7 @@
   <link name="${namespace}/base_link">
       <inertial>
-        <mass value="6.64" />
+        <mass value="8.26" />
         <inertia ixx="0.044958" ixy="0.002614" ixz="0.019172" iyy="0.254345" iyz="0.000036" izz="0.233503" />
-        <origin xyz="-0.37 0 0" rpy="0 0 0" /> <!-- -0.33 -->
+        <origin xyz="-0.346 0 -0.021" rpy="0 0 0" /> <!-- -0.346 for 8.26kg // -0.33 for 6.64kg -->
       </inertial>
       <visual>
@@ -93,7 +93,7 @@
     <parent link="${namespace}/base_link" />
     <child link="${namespace}/wing_left" />
-    <origin xyz="-0.377 0.12 0.114" rpy="0 0 0" />
-    <axis xyz="0 1 0" />
-    <limit upper="0.0" lower="-1.57" effort="10" velocity="20"/>
+    <origin xyz="-0.377 0.12 0.114" rpy="0 -0.7854 0" />
+    <axis xyz="0 -1 0" />
+    <limit upper="0.7854" lower="-0.7854" effort="10" velocity="20"/>
     <dynamics damping="0.2" friction="0" />
   </joint>
@@ -123,7 +123,7 @@
     <parent link="${namespace}/base_link" />
     <child link="${namespace}/wing_right" />
-    <origin xyz="-0.377 -0.12 0.114" rpy="0 0 0" />
-    <axis xyz="0 1 0" />
-    <limit upper="0.0" lower="-1.57" effort="10" velocity="20"/>
+    <origin xyz="-0.377 -0.12 0.114" rpy="0 -0.7854 0" />
+    <axis xyz="0 -1 0" />
+    <limit upper="0.7854" lower="-0.7854" effort="10" velocity="20"/>
     <dynamics damping="0.2" friction="0" />
   </joint>
@@ -156,5 +156,5 @@
     <parent link="${namespace}/wing_left" />
     <child link="${namespace}/aileron_left" />
-    <limit upper="0.53" lower="-0.53" effort="10" velocity="20"/>
+    <limit upper="0.192" lower="-0.192" effort="10" velocity="20"/>
   </joint>
   <link name="${namespace}/aileron_left">
@@ -178,5 +178,5 @@
     <parent link="${namespace}/wing_right" />
     <child link="${namespace}/aileron_right" />
-    <limit upper="0.53" lower="-0.53" effort="10" velocity="20"/>
+    <limit upper="0.192" lower="-0.192" effort="10" velocity="20"/>
   </joint>
   <link name="${namespace}/aileron_right">
@@ -243,5 +243,5 @@
   <!-- Elevator -->
   <joint name="${namespace}/elevator_joint" type="revolute">
-    <origin xyz="-1.335 0 0.0" rpy="0 0 0" />
+    <origin xyz="-1.347 0 0.0" rpy="0 0 0" />
     <axis xyz="0 1 0" />
     <parent link="${namespace}/base_link" />
@@ -255,5 +255,5 @@
     </inertial>
     <visual>
-      <origin xyz="1.335 0 0" rpy="0 0 ${pi/2}" />
+      <origin xyz="1.347 0 0" rpy="0 0 ${pi/2}" />
       <geometry>
           <mesh filename="package://rotors_description/meshes/IGNIS/SCINTILLA/Elevator.stl" scale="0.001 0.001 0.001" />
@@ -266,5 +266,5 @@
   <!-- Propellers -->
   <joint name="${namespace}/propeller_front_left_left_joint" type="continuous">
-    <origin xyz="0.087 0.778 0" rpy="0 ${0.5*pi} 0" />
+    <origin xyz="0.126 0.778 -0.019" rpy="0 ${0.5*pi} 0" />
     <axis xyz="0 0 1" />
     <parent link="${namespace}/wing_left" />
@@ -293,5 +293,5 @@
   </gazebo>
   <joint name="${namespace}/propeller_front_left_joint" type="continuous">
-    <origin xyz="0.087 0.261 0" rpy="0 ${0.5*pi} 0" />
+    <origin xyz="0.126 0.261 -0.019" rpy="0 ${0.5*pi} 0" />
     <axis xyz="0 0 1" />
     <parent link="${namespace}/wing_left" />
@@ -320,5 +320,5 @@
   </gazebo>
   <joint name="${namespace}/propeller_front_right_joint" type="continuous">
-    <origin xyz="0.087 -0.261 0" rpy="0 ${0.5*pi} 0" />
+    <origin xyz="0.126 -0.261 -0.019" rpy="0 ${0.5*pi} 0" />
     <axis xyz="0 0 1" />
     <parent link="${namespace}/wing_right" />
@@ -347,5 +347,5 @@
   </gazebo>
   <joint name="${namespace}/propeller_front_right_right_joint" type="continuous">
-    <origin xyz="0.087 -0.778 0" rpy="0 ${0.5*pi} 0" />
+    <origin xyz="0.126 -0.778 -0.019" rpy="0 ${0.5*pi} 0" />
     <axis xyz="0 0 1" />
     <parent link="${namespace}/wing_right" />
@@ -374,5 +374,5 @@
   </gazebo>
   <joint name="${namespace}/propeller_back_joint" type="continuous">
-    <origin xyz="-1.39 0 0.02" rpy="0 0 0" />
+    <origin xyz="-1.39 0 0.053" rpy="0 0 0" />
     <axis xyz="0 0 1" />
     <parent link="${namespace}/base_link" />
@@ -407,5 +407,5 @@
         <linkNameRef>${namespace}/wing_left</linkNameRef>
         <linkNameAct>${namespace}/base_link</linkNameAct>
-        <cp>0.087 0.778 0</cp>
+        <cp>0.126 0.778 -0.019</cp>
         <axisPosRot>-1 0 0</axisPosRot>
         <turnDir>cw</turnDir>
@@ -424,5 +424,5 @@
         <linkNameRef>${namespace}/wing_left</linkNameRef>
         <linkNameAct>${namespace}/base_link</linkNameAct>
-        <cp>0.087 0.261 0</cp>
+        <cp>0.126 0.261 -0.019</cp>
         <axisPosRot>1 0 0</axisPosRot>
         <turnDir>ccw</turnDir>
@@ -441,5 +441,5 @@
         <linkNameRef>${namespace}/wing_right</linkNameRef>
         <linkNameAct>${namespace}/base_link</linkNameAct>
-        <cp>0.087 -0.261 0</cp>
+        <cp>0.126 -0.261 -0.019</cp>
         <axisPosRot>-1 0 0</axisPosRot>
         <turnDir>cw</turnDir>
@@ -458,5 +458,5 @@
         <linkNameRef>${namespace}/wing_right</linkNameRef>
         <linkNameAct>${namespace}/base_link</linkNameAct>
-        <cp>0.087 -0.778 0</cp>
+        <cp>0.126 -0.778 -0.019</cp>
         <axisPosRot>1 0 0</axisPosRot>
         <turnDir>ccw</turnDir>
@@ -475,7 +475,7 @@
         <linkNameRef>${namespace}/base_link</linkNameRef>
         <linkNameAct>${namespace}/base_link</linkNameAct>
-        <cp>-1.39 0 0.02</cp>
+        <cp>-1.39 0 0.053</cp>
         <axisPosRot>0 0 1</axisPosRot>
-        <turnDir>ccw</turnDir> <!-- !!! -->
+        <turnDir>ccw</turnDir>
         <speedRefTopic>propeller_back_ref</speedRefTopic>
         <propParamsYAML>${yaml_path}/Scintilla_tail_prop.yaml</propParamsYAML>
@@ -524,7 +524,7 @@
           <upward>0 0 1</upward>
           <cp>0 0.25 -0.005</cp>
-          <seg_area>0.06</seg_area>
+          <seg_area>0.03</seg_area>
           <seg_chord>0.1</seg_chord>
-          <aeroParamsYAML>${yaml_path}/Scintilla_wing_airfoil.yaml</aeroParamsYAML> <!-- !!! -->
+          <aeroParamsYAML>${yaml_path}/Scintilla_tail_airfoil.yaml</aeroParamsYAML>
           <wind name="wind">
             <topic>wind_base_link</topic>
@@ -537,7 +537,7 @@
           <upward>0 0 1</upward>
           <cp>0 -0.25 -0.005</cp>
-          <seg_area>0.06</seg_area>
+          <seg_area>0.03</seg_area>
           <seg_chord>0.1</seg_chord>
-          <aeroParamsYAML>${yaml_path}/Scintilla_wing_airfoil.yaml</aeroParamsYAML> <!-- !!! -->
+          <aeroParamsYAML>${yaml_path}/Scintilla_tail_airfoil.yaml</aeroParamsYAML>
           <wind name="wind">
             <topic>wind_base_link</topic>
@@ -549,5 +549,5 @@
           <forward>1 0 0</forward>
           <upward>0 1 0</upward>
-          <cp>-1.17 0.0 0.07</cp>
+          <cp>-1.25 0.0 0.07</cp>
           <seg_area>0.0225</seg_area>
           <seg_chord>0.15</seg_chord>
@@ -570,5 +570,5 @@
         <forward>1 0 0</forward>
         <upward>0 0 1</upward>
-        <cp>0.0 1.0215 0.0</cp>
+        <cp>0.0173 1.0215 -0.01</cp>
         <seg_area>0.006</seg_area>
         <seg_chord>0.208</seg_chord>
@@ -591,5 +591,5 @@
         <forward>1 0 0</forward>
         <upward>0 0 1</upward>
-        <cp>0.0 0.7775 0.0</cp>
+        <cp>0.0173 0.7775 -0.01</cp>
         <seg_area>0.095</seg_area>
         <seg_chord>0.208</seg_chord>
@@ -615,5 +615,5 @@
         <forward>1 0 0</forward>
         <upward>0 0 1</upward>
-        <cp>0.0 0.5190 0.0</cp>
+        <cp>0.0173 0.5190 -0.01</cp>
         <seg_area>0.012</seg_area>
         <seg_chord>0.208</seg_chord>
@@ -636,5 +636,5 @@
         <forward>1 0 0</forward>
         <upward>0 0 1</upward>
-        <cp>0.0 0.2605 0.0</cp>
+        <cp>0.0173 0.2605 -0.01</cp>
         <seg_area>0.095</seg_area>
         <seg_chord>0.208</seg_chord>
@@ -660,5 +660,5 @@
         <forward>1 0 0</forward>
         <upward>0 0 1</upward>
-        <cp>0.0 0.0165 0.0</cp>
+        <cp>0.0173 0.0165 -0.01</cp>
         <seg_area>0.006</seg_area>
         <seg_chord>0.208</seg_chord>
@@ -681,5 +681,5 @@
         <forward>1 0 0</forward>
         <upward>0 0 1</upward>
-        <cp>0.0 -0.0165 0.0</cp>
+        <cp>0.0173 -0.0165 -0.01</cp>
         <seg_area>0.006</seg_area>
         <seg_chord>0.208</seg_chord>
@@ -702,5 +702,5 @@
         <forward>1 0 0</forward>
         <upward>0 0 1</upward>
-        <cp>0.0 -0.2605 0.0</cp>
+        <cp>0.0173 -0.2605 -0.01</cp>
         <seg_area>0.095</seg_area>
         <seg_chord>0.208</seg_chord>
@@ -726,5 +726,5 @@
         <forward>1 0 0</forward>
         <upward>0 0 1</upward>
-        <cp>0.0 -0.5190 0.0</cp>
+        <cp>0.0173 -0.5190 -0.01</cp>
         <seg_area>0.012</seg_area>
         <seg_chord>0.208</seg_chord>
@@ -747,5 +747,5 @@
         <forward>1 0 0</forward>
         <upward>0 0 1</upward>
-        <cp>0.0 -0.7775 0.0</cp>
+        <cp>0.0173 -0.7775 -0.01</cp>
         <seg_area>0.095</seg_area>
         <seg_chord>0.208</seg_chord>
@@ -771,5 +771,5 @@
         <forward>1 0 0</forward>
         <upward>0 0 1</upward>
-        <cp>0.0 -1.0215 0.0</cp>
+        <cp>0.0173 -1.0215 -0.01</cp>
         <seg_area>0.006</seg_area>
         <seg_chord>0.208</seg_chord>
@@ -815,6 +815,6 @@
       <actuatorsPubTopic>/command/motor_speed</actuatorsPubTopic>
       <linkName>${namespace}/base_link</linkName> <!-- reference link frame for airspeed and baro alt-->
-      <pitotPos>0 0 0</pitotPos>           <!-- pitot position wrt reference link -->
-      <baroPos>0 0 0</baroPos>            <!-- baro position wrt reference link -->
+      <pitotPos>-0.417 0.0 -0.008</pitotPos>           <!-- pitot position wrt reference link -->
+      <baroPos>-0.417 0.0 -0.008</baroPos>            <!-- baro position wrt reference link -->
       <wind name="wind">                          <!-- include wind in airspeed measurement -->
         <topic>wind_base_link</topic>
@@ -913,6 +913,6 @@
         <channel name="wing_left">
            <input_index>8</input_index>
-           <input_offset>1</input_offset>
-           <input_scaling>-${1.57*0.5}</input_scaling>
+           <input_offset>0</input_offset>
+           <input_scaling>0.7854</input_scaling>
            <zero_position_disarmed>0</zero_position_disarmed>
            <zero_position_armed>0</zero_position_armed>
@@ -925,6 +925,6 @@
         <channel name="wing_right">
            <input_index>8</input_index>
-           <input_offset>1</input_offset>
-           <input_scaling>-${1.57*0.5}</input_scaling>
+           <input_offset>0</input_offset>
+           <input_scaling>0.7854</input_scaling>
            <zero_position_disarmed>0</zero_position_disarmed>
            <zero_position_armed>0</zero_position_armed>
@@ -938,5 +938,5 @@
           <input_index>9</input_index>
           <input_offset>0</input_offset>
-          <input_scaling>-0.53</input_scaling>
+          <input_scaling>-0.192</input_scaling>
           <zero_position_disarmed>0</zero_position_disarmed>
           <zero_position_armed>0</zero_position_armed>
@@ -951,5 +951,5 @@
           <input_index>10</input_index>
           <input_offset>0</input_offset>
-          <input_scaling>0.53</input_scaling>
+          <input_scaling>0.192</input_scaling>
           <zero_position_disarmed>0</zero_position_disarmed>
           <zero_position_armed>0</zero_position_armed>
