Commit message: Scintilla does not want to be controlled yet

File: rotors_simulator/rotors_description/urdf/SCINTILLA_01.xacro (robot description, xacro)
@@ -416,5 +416,5 @@
         <tauUp>0.075</tauUp>
         <tauDown>0.15</tauDown>
-        <rdpsMax>2039</rdpsMax> <!-- !!! -->
+        <rdpsMax>633</rdpsMax>
         <slpstrTopic>propeller_front_left_left_slpstr</slpstrTopic>
         <visTopic>propeller_front_left_left_vis</visTopic>
@@ -433,5 +433,5 @@
         <tauUp>0.075</tauUp>
         <tauDown>0.15</tauDown>
-        <rdpsMax>2039</rdpsMax> <!-- !!! -->
+        <rdpsMax>633</rdpsMax>
         <slpstrTopic>propeller_front_left_slpstr</slpstrTopic>
         <visTopic>propeller_front_left_vis</visTopic>
@@ -450,5 +450,5 @@
         <tauUp>0.075</tauUp>
         <tauDown>0.15</tauDown>
-        <rdpsMax>2039</rdpsMax> <!-- !!! -->
+        <rdpsMax>633</rdpsMax>
         <slpstrTopic>propeller_front_right_slpstr</slpstrTopic>
         <visTopic>propeller_front_right_vis</visTopic>
@@ -467,5 +467,5 @@
         <tauUp>0.075</tauUp>
         <tauDown>0.15</tauDown>
-        <rdpsMax>2039</rdpsMax> <!-- !!! -->
+        <rdpsMax>633</rdpsMax>
         <slpstrTopic>propeller_front_right_right_slpstr</slpstrTopic>
         <visTopic>propeller_front_right_right_vis</visTopic>
@@ -484,5 +484,5 @@
         <tauUp>0.05</tauUp>
         <tauDown>0.1</tauDown>
-        <rdpsMax>5183</rdpsMax> <!-- !!! -->
+        <rdpsMax>1215</rdpsMax>
         <slpstrTopic>propeller_back_slpstr</slpstrTopic>
         <visTopic>propeller_back_vis</visTopic>
@@ -826,5 +826,5 @@
           <input_index>0</input_index>
           <input_offset>1</input_offset>
-          <input_scaling>1010</input_scaling> <!-- !!! -->
+          <input_scaling>316</input_scaling>
           <zero_position_disarmed>0</zero_position_disarmed>
           <zero_position_armed>0</zero_position_armed>
@@ -844,5 +844,5 @@
           <input_index>1</input_index>
           <input_offset>1</input_offset>
-          <input_scaling>1010</input_scaling> <!-- !!! -->
+          <input_scaling>316</input_scaling>
           <zero_position_disarmed>0</zero_position_disarmed>
           <zero_position_armed>0</zero_position_armed>
@@ -862,5 +862,5 @@
           <input_index>2</input_index>
           <input_offset>1</input_offset>
-          <input_scaling>1010</input_scaling> <!-- !!! -->
+          <input_scaling>316</input_scaling>
           <zero_position_disarmed>0</zero_position_disarmed>
           <zero_position_armed>0</zero_position_armed>
@@ -880,5 +880,5 @@
           <input_index>3</input_index>
           <input_offset>1</input_offset>
-          <input_scaling>1010</input_scaling> <!-- !!! -->
+          <input_scaling>316</input_scaling>
           <zero_position_disarmed>0</zero_position_disarmed>
           <zero_position_armed>0</zero_position_armed>
@@ -898,5 +898,5 @@
           <input_index>4</input_index>
           <input_offset>1</input_offset>
-          <input_scaling>2580</input_scaling> <!-- !!! -->
+          <input_scaling>607</input_scaling>
           <zero_position_disarmed>0</zero_position_disarmed>
           <zero_position_armed>0</zero_position_armed>
@@ -914,5 +914,5 @@
         </channel>
         <channel name="wing_left">
-           <input_index>5</input_index>
+           <input_index>10</input_index>
            <input_offset>0</input_offset>
            <input_scaling>-1.57</input_scaling>
@@ -926,5 +926,5 @@
         </channel>
         <channel name="wing_right">
-           <input_index>5</input_index>
+           <input_index>10</input_index>
            <input_offset>0</input_offset>
            <input_scaling>-1.57</input_scaling>
@@ -938,5 +938,5 @@
         </channel>
         <channel name="aileron_left">
-          <input_index>6</input_index>
+          <input_index>11</input_index>
           <input_offset>0</input_offset>
           <input_scaling>0.53</input_scaling>
@@ -951,5 +951,5 @@
         </channel>
         <channel name="aileron_right">
-          <input_index>7</input_index>
+          <input_index>12</input_index>
           <input_offset>0</input_offset>
           <input_scaling>-0.53</input_scaling>
@@ -964,5 +964,5 @@
         </channel>
         <channel name="elevator">
-          <input_index>8</input_index>
+          <input_index>13</input_index>
           <input_offset>0</input_offset>
           <input_scaling>-1.57</input_scaling>
@@ -976,5 +976,5 @@
         </channel>
         <channel name="rudder">
-          <input_index>9</input_index>
+          <input_index>14</input_index>
           <input_offset>0</input_offset>
           <input_scaling>-0.53</input_scaling>

File: rotors_simulator/rotors_description/urdf/cl84b.xacro (robot description, xacro)
@@ -139,4 +139,23 @@
      <material>Gazebo/Grey</material>
   </gazebo>
+  <joint name="${namespace}/pitot" type="fixed">
+     <origin xyz="0.15 0 -0.08" rpy="0 0 0" />
+     <parent link="${namespace}/base_link" />
+     <child link="${namespace}/pitot" />
+  </joint>
+  <link name="${namespace}/pitot">
+     <inertial>
+        <mass value="0.001" />
+        <xacro:box_inertia x="0.001" y="0.001" z="0.001" mass="0.001" />
+     </inertial>
+     <visual>
+        <geometry>
+           <mesh filename="package://rotors_description/meshes/techpod_X_flex/pitot_tube.stl" scale="1 1 1" />
+        </geometry>
+     </visual>
+  </link>
+  <gazebo reference="${namespace}/pitot">
+     <material>Gazebo/Grey</material>
+  </gazebo>
   <!-- Wing -->
   <joint name="${namespace}/wing_joint" type="revolute">
@@ -399,14 +418,14 @@
         <windLayer>
           <layer name="layer1">
-            <altitude>10</altitude>
-            <windMeanNED>-2 0 0</windMeanNED>
+            <altitude>0.5</altitude>
+            <windMeanNED>-3 -2 0</windMeanNED>
           </layer>
           <layer name="layer2">
             <altitude>25</altitude>
-            <windMeanNED>-3 0 0</windMeanNED>
+            <windMeanNED>-3 -2 0</windMeanNED>
           </layer>
           <layer name="layer3">
             <altitude>35</altitude>
-            <windMeanNED>-10 0 0</windMeanNED>
+            <windMeanNED>-3 -2 0</windMeanNED>
           </layer>
         </windLayer>
@@ -417,9 +436,9 @@
           </query>
         </findWind>
-        <lambdaMin>10</lambdaMin>
+        <lambdaMin>5</lambdaMin>
         <lengthScale>725</lengthScale>
         <fourierNNN>7 7 7</fourierNNN>
-        <sigma>2</sigma>
-        <trnspVelTurbNED>5 0 0</trnspVelTurbNED>
+        <sigma>4</sigma>
+        <trnspVelTurbNED>-3 -2 0</trnspVelTurbNED>
       </plugin>
     </gazebo>
@@ -725,4 +744,37 @@
     </plugin>
   </gazebo>
+  <!-- Flow angle vanes -->
+  <xacro:angle_vane robot_namespace="${namespace}"
+     vane_name="alpha_1"
+     type="alpha"
+     chord="0.02"
+     arm_cp="0.05"
+     mass_vane="0.02"
+     parent="${namespace}/base_link"
+     wind_topic="wind_base_link"
+     color="Grey">
+     <origin xyz="0.60 0.02 0.1" rpy="0 0 0" /><!-- Joint origin -->
+     <xacro:box_inertia x="0.1" y="0.02" z="0.02" mass="0.02" />
+  </xacro:angle_vane>
+  <xacro:angle_vane robot_namespace="${namespace}"
+     vane_name="beta_1"
+     type="beta"
+     chord="0.02"
+     arm_cp="0.05"
+     mass_vane="0.02"
+     parent="${namespace}/base_link"
+     wind_topic="wind_base_link"
+     color="Grey">
+     <origin xyz="0.60 0 0.12" rpy="0 0 0" /><!-- Joint origin -->
+     <xacro:box_inertia x="0.1" y="0.02" z="0.02" mass="0.02" />
+  </xacro:angle_vane>
+  <gazebo>
+     <plugin filename="librotors_gazebo_vane_plugin.so" name="alpha_1_vane_plugin">
+        <robotNamespace>${namespace}</robotNamespace>
+        <alphaJoint>${namespace}/alpha_1_joint</alphaJoint>
+        <betaJoint>${namespace}/beta_1_joint</betaJoint>
+        <vaneTopic>vanes</vaneTopic>
+     </plugin>
+  </gazebo>
   <gazebo>
     <plugin filename="librotors_gazebo_mavlink_interface.so" name="gazebo_mavlink_interface">
@@ -735,4 +787,5 @@
       <lidarSubTopic>/lidar_lite_v3</lidarSubTopic>
       <opticalFlowSubTopic></opticalFlowSubTopic>
+      <vaneSubTopic>/vanes</vaneSubTopic>
       <mavlink_addr>INADDR_ANY</mavlink_addr>
       <mavlink_udp_port>14560</mavlink_udp_port>
@@ -749,6 +802,6 @@
       <actuatorsPubTopic>/command/motor_speed</actuatorsPubTopic>
       <linkName>${namespace}/base_link</linkName> <!-- reference link frame for airspeed and baro alt-->
-      <pitotPos>0 0 0</pitotPos>           <!-- pitot position wrt reference link -->
-      <baroPos>0 0 0</baroPos>            <!-- baro position wrt reference link -->
+      <pitotPos>0.6 0 0.1</pitotPos>                  <!-- pitot position wrt reference link -->
+      <baroPos>0.3 0 0.1</baroPos>                    <!-- baro position wrt reference link -->
       <wind name="wind">                          <!-- include wind in airspeed measurement -->
         <topic>wind_base_link</topic>
@@ -896,5 +949,5 @@
          </servo_params>
          <joint_name>${namespace}/wing_joint</joint_name>
-      </channel><!---->
+      </channel>
     </control_channels>
   </plugin>

Commit message: Update with minor changes to cg position

File: rotors_simulator/rotors_description/urdf/SCINTILLA_01.xacro (robot description, xacro)
@@ -71,5 +71,5 @@
         <mass value="8.26" />
         <inertia ixx="0.044958" ixy="0.002614" ixz="0.019172" iyy="0.254345" iyz="0.000036" izz="0.233503" />
-        <origin xyz="-0.346 0 -0.021" rpy="0 0 0" /> <!-- -0.346 for 8.26kg // -0.33 for 6.64kg -->
+        <origin xyz="-0.346 0 -0.02" rpy="0 0 0" /> <!-- -0.346 0 -0.0196 for 8.26kg // -0.33 0 -0.0224 for 6.64kg -->
       </inertial>
       <visual>

File: rotors_simulator/rotors_description/urdf/SCINTILLA_01_base.xacro (robot description, xacro)
@@ -39,5 +39,5 @@
     enable_delay = "false">
     <xacro:cube_inertia l="0.02" mass="0.015" />
-    <origin xyz="-0.417 0 0" rpy="0 0 0" />
+    <origin xyz="-0.417 0 -0.008" rpy="0 0 0" />
   </xacro:gps_plugin_macro>
   <xacro:gps_plugin_macro
@@ -54,5 +54,5 @@
     enable_delay = "false">
     <xacro:cube_inertia l="0.02" mass="0.001" />
-    <origin xyz="-0.417 0 0" rpy="0 0 0" />
+    <origin xyz="-0.417 0 -0.008" rpy="0 0 0" />
   </xacro:gps_plugin_macro>
   <xacro:camera_macro_2
@@ -73,5 +73,5 @@
     <mesh filename="package://rotors_description/meshes/vi_camera.dae" scale="1 1 1" />
     <xacro:cube_inertia l="0.02" mass="0.01" />
-    <origin xyz="-0.417 0 0" rpy="0 0.2 0" />
+    <origin xyz="-0.417 0 -0.008" rpy="0 0 0" />
   </xacro:camera_macro_2>
 </robot>

Commit message: slightly modfied scintilla (smoother stall, c_ld aileron adjusted), sigmoid non-stall/stall mixing, wing-tilt 0-pi/2 working

File: rotors_simulator/rotors_description/urdf/SCINTILLA_01.xacro (robot description, xacro)
@@ -93,7 +93,7 @@
     <parent link="${namespace}/base_link" />
     <child link="${namespace}/wing_left" />
-    <origin xyz="-0.377 0.12 0.114" rpy="0 -0.7854 0" />
+    <origin xyz="-0.377 0.12 0.114" rpy="0 0 0" />
     <axis xyz="0 -1 0" />
-    <limit upper="0.7854" lower="-0.7854" effort="10" velocity="20"/>
+    <limit lower="0" upper="1.57" effort="10" velocity="20"/>
     <dynamics damping="0.2" friction="0" />
   </joint>
@@ -123,7 +123,7 @@
     <parent link="${namespace}/base_link" />
     <child link="${namespace}/wing_right" />
-    <origin xyz="-0.377 -0.12 0.114" rpy="0 -0.7854 0" />
+    <origin xyz="-0.377 -0.12 0.114" rpy="0 0 0" />
     <axis xyz="0 -1 0" />
-    <limit upper="0.7854" lower="-0.7854" effort="10" velocity="20"/>
+    <limit lower="0" upper="1.57" effort="10" velocity="20"/>
     <dynamics damping="0.2" friction="0" />
   </joint>
@@ -516,5 +516,5 @@
     <plugin filename="librotors_gazebo_aerodynamics_plugin.so" name="aerodynamics_plugin">
       <robotNamespace>${namespace}</robotNamespace>
-      <aeroForcesVis>aero_force_vis_1</aeroForcesVis>
+      <aeroForcesVis>aero_force_vis_tail</aeroForcesVis>
       <airfoil>
         <segment name="EL">
@@ -563,5 +563,5 @@
     <plugin filename="librotors_gazebo_aerodynamics_plugin.so" name="aerodynamics_plugin">
       <robotNamespace>${namespace}</robotNamespace>
-      <aeroForcesVis>aero_force_vis_1</aeroForcesVis>
+      <aeroForcesVis>aero_force_vis_wing</aeroForcesVis>
       <airfoil>
       <segment name="WL1">
@@ -580,5 +580,5 @@
           <cs name="aileron_left">
               <controlJoint>${namespace}/aileron_left_joint</controlJoint>
-              <radToCLift>2</radToCLift>
+              <radToCLift>1.2</radToCLift>
               <radToCDrag>0.0</radToCDrag>
               <radToCPitch>0.0</radToCPitch>
@@ -598,5 +598,5 @@
           <cs name="aileron_left">
               <controlJoint>${namespace}/aileron_left_joint</controlJoint>
-              <radToCLift>2</radToCLift>
+              <radToCLift>1.2</radToCLift>
               <radToCDrag>0.0</radToCDrag>
               <radToCPitch>0.0</radToCPitch>
@@ -625,5 +625,5 @@
           <cs name="aileron_left">
               <controlJoint>${namespace}/aileron_left_joint</controlJoint>
-              <radToCLift>2</radToCLift>
+              <radToCLift>1.2</radToCLift>
               <radToCDrag>0.0</radToCDrag>
               <radToCPitch>0.0</radToCPitch>
@@ -643,5 +643,5 @@
           <cs name="aileron_left">
               <controlJoint>${namespace}/aileron_left_joint</controlJoint>
-              <radToCLift>2</radToCLift>
+              <radToCLift>1.2</radToCLift>
               <radToCDrag>0.0</radToCDrag>
               <radToCPitch>0.0</radToCPitch>
@@ -670,5 +670,5 @@
           <cs name="aileron_left">
               <controlJoint>${namespace}/aileron_left_joint</controlJoint>
-              <radToCLift>2</radToCLift>
+              <radToCLift>1.2</radToCLift>
               <radToCDrag>0.0</radToCDrag>
               <radToCPitch>0.0</radToCPitch>
@@ -691,5 +691,5 @@
           <cs name="aileron_right">
               <controlJoint>${namespace}/aileron_right_joint</controlJoint>
-              <radToCLift>2</radToCLift>
+              <radToCLift>1.2</radToCLift>
               <radToCDrag>0.0</radToCDrag>
               <radToCPitch>0.0</radToCPitch>
@@ -709,5 +709,5 @@
           <cs name="aileron_right">
               <controlJoint>${namespace}/aileron_right_joint</controlJoint>
-              <radToCLift>2</radToCLift>
+              <radToCLift>1.2</radToCLift>
               <radToCDrag>0.0</radToCDrag>
               <radToCPitch>0.0</radToCPitch>
@@ -736,5 +736,5 @@
           <cs name="aileron_right">
               <controlJoint>${namespace}/aileron_right_joint</controlJoint>
-              <radToCLift>2</radToCLift>
+              <radToCLift>1.2</radToCLift>
               <radToCDrag>0.0</radToCDrag>
               <radToCPitch>0.0</radToCPitch>
@@ -754,5 +754,5 @@
           <cs name="aileron_right">
               <controlJoint>${namespace}/aileron_right_joint</controlJoint>
-              <radToCLift>2</radToCLift>
+              <radToCLift>1.2</radToCLift>
               <radToCDrag>0.0</radToCDrag>
               <radToCPitch>0.0</radToCPitch>
@@ -781,5 +781,5 @@
           <cs name="aileron_right">
               <controlJoint>${namespace}/aileron_right_joint</controlJoint>
-              <radToCLift>2</radToCLift>
+              <radToCLift>1.2</radToCLift>
               <radToCDrag>0.0</radToCDrag>
               <radToCPitch>0.0</radToCPitch>
@@ -913,5 +913,5 @@
         <channel name="wing_left">
            <input_index>8</input_index>
-           <input_offset>0</input_offset>
+           <input_offset>1</input_offset>
            <input_scaling>0.7854</input_scaling>
            <zero_position_disarmed>0</zero_position_disarmed>
@@ -925,5 +925,5 @@
         <channel name="wing_right">
            <input_index>8</input_index>
-           <input_offset>0</input_offset>
+           <input_offset>1</input_offset>
            <input_scaling>0.7854</input_scaling>
            <zero_position_disarmed>0</zero_position_disarmed>

Commit message: Final Presentation update

File: rotors_simulator/rotors_description/urdf/SCINTILLA_01.xacro (robot description, xacro)
@@ -1,5 +1,5 @@
 <?xml version="1.0" encoding="UTF-8"?>
 <!--
-  Copyright 2016 Pavel Vechersky, ASL, ETH Zurich, Switzerland
+  Copyright 2016 Pavel Vechersky, ASL, ETH Zurich, Switzerland !!!
   Licensed under the Apache License, Version 2.0 (the "License");
   you may not use this file except in compliance with the License.
@@ -66,10 +66,10 @@
   </xacro:property>
   <xacro:include filename="$(find rotors_description)/urdf/fixed_wing_X_base.xacro" />
-  <!-- Fuselage - Ineritas and Masses need to be checked -->
+  <!-- Fuselage -->
   <link name="${namespace}/base_link">
       <inertial>
         <mass value="8.26" />
         <inertia ixx="0.044958" ixy="0.002614" ixz="0.019172" iyy="0.254345" iyz="0.000036" izz="0.233503" />
-        <origin xyz="-0.346 0 -0.02" rpy="0 0 0" /> <!-- -0.346 0 -0.0196 for 8.26kg // -0.33 0 -0.0224 for 6.64kg -->
+        <origin xyz="-0.346 0 -0.02" rpy="0 0 0" /> <!-- -0.346 0 -0.0196 for 8.26kg / -0.353 for CG shift of -0.005 // -0.33 0 -0.0224 for 6.64kg -->
       </inertial>
       <visual>
@@ -516,5 +516,5 @@
     <plugin filename="librotors_gazebo_aerodynamics_plugin.so" name="aerodynamics_plugin">
       <robotNamespace>${namespace}</robotNamespace>
-      <aeroForcesVis>aero_force_vis_1</aeroForcesVis>
+      <aeroForcesVis>aero_force_vis_tail</aeroForcesVis>
       <airfoil>
         <segment name="EL">
@@ -563,5 +563,5 @@
     <plugin filename="librotors_gazebo_aerodynamics_plugin.so" name="aerodynamics_plugin">
       <robotNamespace>${namespace}</robotNamespace>
-      <aeroForcesVis>aero_force_vis_1</aeroForcesVis>
+      <aeroForcesVis>aero_force_vis_wing</aeroForcesVis>
       <airfoil>
       <segment name="WL1">
@@ -580,5 +580,5 @@
           <cs name="aileron_left">
               <controlJoint>${namespace}/aileron_left_joint</controlJoint>
-              <radToCLift>2</radToCLift>
+              <radToCLift>1.2</radToCLift>
               <radToCDrag>0.0</radToCDrag>
               <radToCPitch>0.0</radToCPitch>
@@ -598,5 +598,5 @@
           <cs name="aileron_left">
               <controlJoint>${namespace}/aileron_left_joint</controlJoint>
-              <radToCLift>2</radToCLift>
+              <radToCLift>1.2</radToCLift>
               <radToCDrag>0.0</radToCDrag>
               <radToCPitch>0.0</radToCPitch>
@@ -625,5 +625,5 @@
           <cs name="aileron_left">
               <controlJoint>${namespace}/aileron_left_joint</controlJoint>
-              <radToCLift>2</radToCLift>
+              <radToCLift>1.2</radToCLift>
               <radToCDrag>0.0</radToCDrag>
               <radToCPitch>0.0</radToCPitch>
@@ -643,5 +643,5 @@
           <cs name="aileron_left">
               <controlJoint>${namespace}/aileron_left_joint</controlJoint>
-              <radToCLift>2</radToCLift>
+              <radToCLift>1.2</radToCLift>
               <radToCDrag>0.0</radToCDrag>
               <radToCPitch>0.0</radToCPitch>
@@ -670,5 +670,5 @@
           <cs name="aileron_left">
               <controlJoint>${namespace}/aileron_left_joint</controlJoint>
-              <radToCLift>2</radToCLift>
+              <radToCLift>1.2</radToCLift>
               <radToCDrag>0.0</radToCDrag>
               <radToCPitch>0.0</radToCPitch>
@@ -691,5 +691,5 @@
           <cs name="aileron_right">
               <controlJoint>${namespace}/aileron_right_joint</controlJoint>
-              <radToCLift>2</radToCLift>
+              <radToCLift>1.2</radToCLift>
               <radToCDrag>0.0</radToCDrag>
               <radToCPitch>0.0</radToCPitch>
@@ -709,5 +709,5 @@
           <cs name="aileron_right">
               <controlJoint>${namespace}/aileron_right_joint</controlJoint>
-              <radToCLift>2</radToCLift>
+              <radToCLift>1.2</radToCLift>
               <radToCDrag>0.0</radToCDrag>
               <radToCPitch>0.0</radToCPitch>
@@ -736,5 +736,5 @@
           <cs name="aileron_right">
               <controlJoint>${namespace}/aileron_right_joint</controlJoint>
-              <radToCLift>2</radToCLift>
+              <radToCLift>1.2</radToCLift>
               <radToCDrag>0.0</radToCDrag>
               <radToCPitch>0.0</radToCPitch>
@@ -754,5 +754,5 @@
           <cs name="aileron_right">
               <controlJoint>${namespace}/aileron_right_joint</controlJoint>
-              <radToCLift>2</radToCLift>
+              <radToCLift>1.2</radToCLift>
               <radToCDrag>0.0</radToCDrag>
               <radToCPitch>0.0</radToCPitch>
@@ -781,5 +781,5 @@
           <cs name="aileron_right">
               <controlJoint>${namespace}/aileron_right_joint</controlJoint>
-              <radToCLift>2</radToCLift>
+              <radToCLift>1.2</radToCLift>
               <radToCDrag>0.0</radToCDrag>
               <radToCPitch>0.0</radToCPitch>
@@ -964,5 +964,5 @@
           <input_index>11</input_index>
           <input_offset>0</input_offset>
-          <input_scaling>-0.53</input_scaling>
+          <input_scaling>0.53</input_scaling>
           <zero_position_disarmed>0</zero_position_disarmed>
           <zero_position_armed>0</zero_position_armed>
