Commit message: IMU changed to configure noise

File: rotors_simulator/rotors_description/urdf/SCINTILLA_01_base.xacro (robot description, xacro)
@@ -17,7 +17,38 @@
   <xacro:include filename="$(find rotors_description)/urdf/SCINTILLA_01.xacro" />
   <!-- Mount an ADIS16448 IMU. -->
-  <xacro:default_imu namespace="${namespace}" parent_link="${namespace}/base_link" >
-    <origin xyz="-0.45 0 0.065" rpy="0 0 0" />  <!-- !!! Where our Pixhawk lies-->
-  </xacro:default_imu>
+  <xacro:imu_plugin_macro
+      namespace="${namespace}"
+      imu_suffix=""
+      parent_link="${namespace}/base_link"
+      imu_topic="imu"
+      mass_imu_sensor="0.015"
+      gyroscope_noise_density="0.0"
+      gyroscope_random_walk="0.0"
+      gyroscope_bias_correlation_time="0.0"
+      gyroscope_turn_on_bias_sigma="0.0"
+      accelerometer_noise_density="0.0"
+      accelerometer_random_walk="0.0"
+      accelerometer_bias_correlation_time="0.0"
+      accelerometer_turn_on_bias_sigma="0.0">
+      <origin xyz="-0.45 0 0.065" rpy="0 0 0" />  <!-- !!! Where our Pixhawk lies-->
+      <xacro:cube_inertia l="0.02" mass="0.015" />
+    </xacro:imu_plugin_macro>
+    <!-- <xacro:imu_plugin_macro
+        namespace="${namespace}"
+        imu_suffix=""
+        parent_link="${namespace}/base_link"
+        imu_topic="imu"
+        mass_imu_sensor="0.015"
+        gyroscope_noise_density="0.0003394"
+        gyroscope_random_walk="0.000038785"
+        gyroscope_bias_correlation_time="1000.0"
+        gyroscope_turn_on_bias_sigma="0.0087"
+        accelerometer_noise_density="0.004"
+        accelerometer_random_walk="0.006"
+        accelerometer_bias_correlation_time="300.0"
+        accelerometer_turn_on_bias_sigma="0.1960">
+        <origin xyz="-0.45 0 0.065" rpy="0 0 0" />
+        <xacro:cube_inertia l="0.02" mass="0.015" />
+      </xacro:imu_plugin_macro> -->
   <!-- Mount a GPS.-->
   <!--<xacro:default_gps
